File: micromouse-main-board/MicromouseV0.0.3.sch (EAGLE design)
At the start: 12 parts

Commit message: got board outline to work
Parts:
- removed U$1, U$2, U$3, U$4, U$5, U$6: EMITTER, chok_boi:EMITTER
- removed U$10: RECEIVER, chok_boi:RECEIVER
- added C_ELF1, C_EM_D1, C_ERF1, C_E_H1: 4.7uF, SparkFun-Capacitors:CAP0603-CAP
- added C_ELF2, C_EM_D2, C_ERF2, C_E_H2: 0.1uF, SparkFun-Capacitors:CAP0603-CAP
- added LEFT_FRONT_EMITTER, U$11, U$13, U$17, U$18, U$19: EMITTER, sfh4550 _ teft4300:EMITTER
- added NMOS1, NMOS2, NMOS3, NMOS4: DMN3150LW, DMN3150LW:DMN3150LW
- added REC_LF, U$20, U$21: RECEIVER, sfh4550 _ teft4300:RECEIVER
- added R_ED1, R_ED2, R_EH1, R_EH2: 5.6, SparkFun-Passives:RESISTOR0603-RES
- added R_ED_PD, R_EH_PD, R_ELF_PD, R_ERF_PD: 47k, SparkFun-Passives:RESISTOR0603-RES
- added R_ELF, R_ERF: 10, SparkFun-Passives:RESISTOR0603-RES
- added R_RLD, R_RLF, R_RLH, R_RRD, R_RRF, R_RRH: 1.8k, SparkFun-Passives:RESISTOR0603-RES
- U$7, U$8, U$9: device chok_boi:RECEIVER -> sfh4550 _ teft4300:RECEIVER
Connections:
- new net A3.3V: REC_LF.C, U$20.C, U$21.C, U$7.C, U$8.C, U$9.C
- new net AGND: R_RLD.1, R_RLF.1, R_RLH.1, R_RRD.1, R_RRF.1, R_RRH.1
- new net D2_EM: R_ED1.2, R_ED2.2, U$17.-
- new net D_EM: U$11.-, U$17.+
- new net EM_D: NMOS2.G, R_ED_PD.2
- new net EM_H: NMOS4.G, R_EH_PD.2
- new net EM_LF: NMOS1.G, R_ELF_PD.2
- new net EM_RF: NMOS3.G, R_ERF_PD.2
- new net H2_EM: R_EH1.2, R_EH2.2, U$19.-
- new net H_EM: U$18.-, U$19.+
- new net LF_EM: LEFT_FRONT_EMITTER.-, R_ELF.2
- new net N$18: NMOS2.D, R_ED1.1, R_ED2.1
- new net N$19: NMOS4.D, R_EH1.1, R_EH2.1
- new net N$5: NMOS3.D, R_ERF.1
- new net N$7: NMOS1.D, R_ELF.1
- new net REC_LD: R_RLD.2, U$7.E
- new net REC_LF: REC_LF.E, R_RLF.2
- new net REC_LH: R_RLH.2, U$21.E
- new net REC_RD: R_RRD.2, U$8.E
- new net REC_RF: R_RRF.2, U$9.E
- new net REC_RH: R_RRH.2, U$20.E
- new net RF_EM: R_ERF.2, U$13.-
- net 5V: now also C_ELF1.1, C_ELF2.1, C_EM_D1.1, C_EM_D2.1, C_ERF1.1, C_ERF2.1, C_E_H1.1, C_E_H2.1, LEFT_FRONT_EMITTER.+, U$11.+, U$13.+, U$18.+
- net GND: now also C_ELF1.2, C_ELF2.2, C_EM_D1.2, C_EM_D2.2, C_ERF1.2, C_ERF2.2, C_E_H1.2, C_E_H2.2, NMOS1.S, NMOS2.S, NMOS3.S, NMOS4.S, R_ED_PD.1, R_EH_PD.1, R_ELF_PD.1, R_ERF_PD.1
Other:
- note added: "Changelog -------------------------------------- 06/08/2019 - Added MCU, board outline and IR sensors and receivers."
- note added: "Note: Enable Pins need to be changed"
- note added: "Notes -------------------------------------- Add product specs and notes on 'Guide' layer Use GND symbol and VCC symbol for ground and power respectively. (Rather than tags)"
- moved on the sheet: CR1
