File: micromouse-main-board/MicromouseV0.0.3.sch (EAGLE design)
At the start: 42 parts

Commit message: updated board
Connections:
- net EM_LF renamed LABEL_ME
Changed lines of the file:
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@@
 </segment>
 </net>
-<net name="EM_LF" class="0">
+<net name="LABEL_ME" class="0">
 <segment>
 <pinref part="R_ELF_PD" gate="G$1" pin="2"/>

Commit message: update
Parts:
- added C1, C2, C3, C4, C7, C8: .1uF, rcl:C-USC0603
- added C5, C6: (no value), rcl:C-USC0603
- added R1: 1k, rcl:R-US_M0805
- added U1: SN74HC151DR, SN74HC151DR:SN74HC151DR
- added U2: DRV8848PWPR, DRV8848PWPR:DRV8848PWPR
- added U3: ACS712ELCTR-20A-T, ACS712ELCTR-20A-T:ACS712ELCTR-20A-T
Connections:
- new net 3V3: C1.1, C2.1, C3.1, C4.1, C7.1, C8.1, CR1.VDDA, CR1.VDD_1, CR1.VDD_2, CR1.VDD_3, CR1.VDD_4, U1.VCC
- new net ADC_IN: CR1.PC3
- new net I2C_SCL: CR1.PB6
- new net I2C_SDA: CR1.PB7
- new net MUX_EN: CR1.PA11, U1.~G
- new net N$21: CR1.VSS_3
- new net N$9: CR1.BOOT0, R1.1
- new net NRST: CR1.NRST
- new net SEL_A: CR1.PA8, U1.A
- new net SEL_B: CR1.PA9, U1.B
- new net SEL_C: CR1.PA10, U1.C
- new net SPI_MISO: CR1.PB14
- new net SPI_MOSI: CR1.PB15
- new net SPI_NSS: CR1.PB12
- new net SPI_SCK: CR1.PB13
- new net SWCLK: CR1.PA14
- new net SWDIO: CR1.PA13
- net GND: now also C1.2, C2.2, C3.2, C4.2, C7.2, C8.2, CR1.VSSA, CR1.VSS_1, CR1.VSS_2, CR1.VSS_4, R1.2, U1.GND
- net REC_LD: now also U1.D1
- net REC_LF: now also U1.D0
- net REC_LH: now also U1.D5
- net REC_RD: now also U1.D2
- net REC_RF: now also U1.D3
- net REC_RH: now also U1.D4
Other:
- note added: "Changelog -------------------------------------- 06/08/2019 - Added MCU, board outline and IR sensors and receivers. 07/17/2019 - Added Motor Driver, MUX for sensor input, Current Sensor, Voltage Sensor, picked GPIO to use for MUX select, picked ADC in to route MUX to."
- note removed: "Changelog -------------------------------------- 06/08/2019 - Added MCU, board outline and IR sensors and receivers."
