File: micromouse-main-board/MicromouseV0.0.3.sch (EAGLE design)
At the start: 54 parts, among them U1 SN74HC151DR, U2 DRV8848PWPR, U3 ACS712ELCTR-20A-T

Commit message: Added debug header
Parts:
- added J1: (no value), SparkFun-Connectors:CONN_04
Connections:
- net 3V3: now also J1.4
- net GND: now also J1.1
- net SWCLK: now also J1.2
- net SWDIO: now also J1.3
Other:
- note added: "Changelog -------------------------------------- 06/08/2019 - Added MCU, board outline and IR sensors and receivers. 07/17/2019 - Added Motor Driver, MUX for sensor input, Current Sensor, picked GPIO to use for MUX select, picked ADC in to route MUX to. 07/18/2019 - Programming/debug header added."
- note added: "PROGRAMMING/DEBUG HEADER"
- note removed: "Changelog -------------------------------------- 06/08/2019 - Added MCU, board outline and IR sensors and receivers. 07/17/2019 - Added Motor Driver, MUX for sensor input, Current Sensor, picked GPIO to use for MUX select, picked ADC in to route MUX to."
Changed lines of the file:
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@@
 <part name="GND17" library="supply1" deviceset="GND" device=""/>
 <part name="GND18" library="supply1" deviceset="GND" device=""/>
+<part name="J1" library="SparkFun-Connectors" library_urn="urn:adsk.eagle:library:513" deviceset="CONN_04" device="" package3d_urn="urn:adsk.eagle:package:38085/1"/>
+<part name="GND19" library="supply1" deviceset="GND" device=""/>
 </parts>
 <sheets>
@@
 --------------------------------------
 06/08/2019 - Added MCU, board outline and IR sensors and receivers.
-07/17/2019 - Added Motor Driver, MUX for sensor input, Current Sensor, picked GPIO to use for MUX select, picked ADC in to route MUX to. </text>
+07/17/2019 - Added Motor Driver, MUX for sensor input, Current Sensor, picked GPIO to use for MUX select, picked ADC in to route MUX to.
+07/18/2019 - Programming/debug header added.</text>
 <text x="429.26" y="210.82" size="2.54" layer="98" font="vector">Note: Enable Pins need to be changed</text>
 <text x="431.8" y="129.54" size="2.54" layer="98" font="vector">Note: Enable Pins need to be changed</text>
@@
 Use GND symbol and VCC symbol for ground and power respectively.
 (Rather than tags)</text>
+<text x="88.9" y="218.44" size="1.778" layer="94">PROGRAMMING/DEBUG HEADER</text>
 </plain>
 <instances>
@@
 <instance part="GND18" gate="1" x="-27.94" y="83.82" smashed="yes">
 <attribute name="VALUE" x="-30.48" y="81.28" size="1.778" layer="96"/>
+</instance>
+<instance part="J1" gate="G$1" x="106.68" y="203.2"/>
+<instance part="GND19" gate="1" x="114.3" y="195.58" smashed="yes">
+<attribute name="VALUE" x="111.76" y="193.04" size="1.778" layer="96"/>
 </instance>
 </instances>
@@
 <wire x1="-22.86" y1="203.2" x2="-25.4" y2="203.2" width="0.1524" layer="91"/>
 </segment>
+<segment>
+<pinref part="J1" gate="G$1" pin="1"/>
+<wire x1="111.76" y1="200.66" x2="114.3" y2="200.66" width="0.1524" layer="91"/>
+<pinref part="GND19" gate="1" pin="GND"/>
+<wire x1="114.3" y1="200.66" x2="114.3" y2="198.12" width="0.1524" layer="91"/>
+</segment>
 </net>
 <net name="5V" class="0">
@@
 <label x="45.72" y="203.2" size="1.778" layer="95" rot="R90"/>
 </segment>
+<segment>
+<pinref part="J1" gate="G$1" pin="2"/>
+<wire x1="111.76" y1="203.2" x2="114.3" y2="203.2" width="0.1524" layer="91"/>
+<label x="114.3" y="203.2" size="1.778" layer="95"/>
+</segment>
 </net>
 <net name="SWDIO" class="0">
@@
 <wire x1="58.42" y1="172.72" x2="63.5" y2="172.72" width="0.1524" layer="91"/>
 <label x="63.5" y="172.72" size="1.778" layer="95"/>
+</segment>
+<segment>
+<pinref part="J1" gate="G$1" pin="3"/>
+<wire x1="111.76" y1="205.74" x2="114.3" y2="205.74" width="0.1524" layer="91"/>
+<label x="114.3" y="205.74" size="1.778" layer="95"/>
 </segment>
 </net>
@@
 <junction x="116.84" y="165.1"/>
 </segment>
-</net>
+<segment>
+<pinref part="J1" gate="G$1" pin="4"/>
+<wire x1="111.76" y1="208.28" x2="114.3" y2="208.28" width="0.1524" layer="91"/>
+<label x="114.3" y="208.28" size="1.778" layer="95"/>
+</segment>
+</net>
