File: micromouse-main-board/MicromouseV0.0.3.brd (EAGLE design)
At the start: 86 x 74 mm, 12 parts

Commit message: got board outline to work
Parts:
- removed U$1, U$2, U$3, U$4, U$5, U$6: EMITTER, chok_boi:EMITTER
- removed U$10: RECEIVER, chok_boi:RECEIVER
- added C_ELF1, C_EM_D1, C_ERF1, C_E_H1: 4.7uF, SparkFun-Capacitors:0603-CAP
- added C_ELF2, C_EM_D2, C_ERF2, C_E_H2: 0.1uF, SparkFun-Capacitors:0603-CAP
- added LEFT_FRONT_EMITTER, U$11, U$13, U$17, U$18, U$19: EMITTER, sfh4550 _ teft4300:EMITTER
- added NMOS1, NMOS2, NMOS3, NMOS4: DMN3150LW, DMN3150LW:DMN3150LW
- added REC_LF, U$20, U$21: RECEIVER, sfh4550 _ teft4300:RECEIVER
- added R_ED1, R_ED2, R_EH1, R_EH2: 5.6, SparkFun-Passives:0603-RES
- added R_ED_PD, R_EH_PD, R_ELF_PD, R_ERF_PD: 47k, SparkFun-Passives:0603-RES
- added R_ELF, R_ERF: 10, SparkFun-Passives:0603-RES
- added R_RLD, R_RLF, R_RLH, R_RRD, R_RRF, R_RRH: 1.8k, SparkFun-Passives:0603-RES
- U$7, U$8, U$9: device chok_boi:RECEIVER -> sfh4550 _ teft4300:RECEIVER
- moved U$12 351.9 mm to (0.00, 37.0), turned to 270 degrees
- moved U$8 350.3 mm to (79.0, 27.0), turned to 220 degrees
- moved U$7 344.6 mm to (79.0, 47.0), turned to 320 degrees
- moved U$9 340.2 mm to (62.0, 10.0), turned to 267 degrees
- moved CR1 66.1 mm to (57.2, 37.1)
Connections:
- new net A3.3V: REC_LF.C, U$20.C, U$21.C, U$7.C, U$8.C, U$9.C
- new net AGND: R_RLD.1, R_RLF.1, R_RLH.1, R_RRD.1, R_RRF.1, R_RRH.1
- new net D2_EM: R_ED1.2, R_ED2.2, U$17.-
- new net D_EM: U$11.-, U$17.+
- new net EM_D: NMOS2.G, R_ED_PD.2
- new net EM_H: NMOS4.G, R_EH_PD.2
- new net EM_LF: NMOS1.G, R_ELF_PD.2
- new net EM_RF: NMOS3.G, R_ERF_PD.2
- new net H2_EM: R_EH1.2, R_EH2.2, U$19.-
- new net H_EM: U$18.-, U$19.+
- new net LF_EM: LEFT_FRONT_EMITTER.-, R_ELF.2
- new net N$18: NMOS2.D, R_ED1.1, R_ED2.1
- new net N$19: NMOS4.D, R_EH1.1, R_EH2.1
- new net N$5: NMOS3.D, R_ERF.1
- new net N$7: NMOS1.D, R_ELF.1
- new net REC_LD: R_RLD.2, U$7.E
- new net REC_LF: REC_LF.E, R_RLF.2
- new net REC_LH: R_RLH.2, U$21.E
- new net REC_RD: R_RRD.2, U$8.E
- new net REC_RF: R_RRF.2, U$9.E
- new net REC_RH: R_RRH.2, U$20.E
- new net RF_EM: R_ERF.2, U$13.-
- net 5V: now also C_ELF1.1, C_ELF2.1, C_EM_D1.1, C_EM_D2.1, C_ERF1.1, C_ERF2.1, C_E_H1.1, C_E_H2.1, LEFT_FRONT_EMITTER.+, U$11.+, U$13.+, U$18.+
- net GND: now also C_ELF1.2, C_ELF2.2, C_EM_D1.2, C_EM_D2.2, C_ERF1.2, C_ERF2.2, C_E_H1.2, C_E_H2.2, NMOS1.S, NMOS2.S, NMOS3.S, NMOS4.S, R_ED_PD.1, R_EH_PD.1, R_ELF_PD.1, R_ERF_PD.1
Routing:
- added copper zone on layer 1, net AGND
- added copper zone on layer 16, net GND
Other:
- board text added: "Notes ----------------------- Bottom layer - GND Add net classes Add power planes Use vector font"
- board text added: "RESET"

Commit message: updated board
Connections:
- net EM_LF renamed LABEL_ME
Other:
- board text added: "(mm)"
Changed lines of the file:
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@@
 <setting verticaltext="up"/>
 </settings>
-<grid distance="0.0125" unitdist="inch" unit="mil" style="lines" multiple="1" display="yes" altdistance="1" altunitdist="mil" altunit="mil"/>
+<grid distance="5" unitdist="mil" unit="mil" style="lines" multiple="1" display="yes" altdistance="1" altunitdist="mil" altunit="mil"/>
 <layers>
 <layer number="1" name="Top" color="4" fill="1" visible="yes" active="yes"/>
@@
 Add power planes
 Use vector font </text>
+<dimension x1="20.066" y1="65.024" x2="19.939" y2="9.017" x3="14.03439375" y3="37.034034375" textsize="1.778" layer="48"/>
+<dimension x1="29.972" y1="35.433" x2="29.972" y2="9.525" x3="19.177" y3="22.479" textsize="1.778" layer="48"/>
+<dimension x1="19.939" y1="0" x2="51.943" y2="0" x3="35.941" y3="-8.763" textsize="1.778" layer="48"/>
+<text x="39.497" y="-7.874" size="1.778" layer="48">(mm)</text>
 </plain>
 <attributes>
@@
 <contactref element="U$12" pad="R_MOTOR_B"/>
 </signal>
-<signal name="EM_LF">
+<signal name="LABEL_ME">
 <contactref element="R_ELF_PD" pad="2"/>
 <contactref element="NMOS1" pad="G"/>

Commit message: update
Parts:
- added C1, C2, C3, C4, C7, C8: .1uF, rcl:C0603
- added C5, C6: (no value), rcl:C0603
- added R1: 1k, rcl:M0805
- added U1: SN74HC151DR, SN74HC151DR:SOIC127P600X175-16N
- added U2: DRV8848PWPR, DRV8848PWPR:SOP65P640X120-17N
- added U3: ACS712ELCTR-20A-T, ACS712ELCTR-20A-T:SOIC127P600X175-8N
Connections:
- net VSS_3 renamed N$21
- removed net VDDA: CR1.13
- removed net VDD_1: CR1.32
- removed net VDD_2: CR1.48
- removed net VDD_3: CR1.64
- removed net VDD_4: CR1.19
- removed net VSSA: CR1.12
- removed net VSS_1: CR1.31
- removed net VSS_2: CR1.47
- removed net VSS_4: CR1.18
- new net 3V3: C1.1, C2.1, C3.1, C4.1, C7.1, C8.1, CR1.13, CR1.19, CR1.32, CR1.48, CR1.64, U1.16
- new net ADC_IN: CR1.11
- new net I2C_SCL: CR1.58
- new net I2C_SDA: CR1.59
- new net MUX_EN: CR1.44, U1.7
- new net N$9: CR1.60, R1.1
- new net NRST: CR1.7
- new net SEL_A: CR1.41, U1.11
- new net SEL_B: CR1.42, U1.10
- new net SEL_C: CR1.43, U1.9
- new net SPI_MISO: CR1.35
- new net SPI_MOSI: CR1.36
- new net SPI_NSS: CR1.33
- new net SPI_SCK: CR1.34
- new net SWCLK: CR1.49
- new net SWDIO: CR1.46
- new net VCC: U3.8
- net GND: now also C1.2, C2.2, C3.2, C4.2, C7.2, C8.2, CR1.12, CR1.18, CR1.31, CR1.47, R1.2, U1.8, U2.13
- net REC_LD: now also U1.3
- net REC_LF: now also U1.4
- net REC_LH: now also U1.14
- net REC_RD: now also U1.2
- net REC_RF: now also U1.1
- net REC_RH: now also U1.15
