File: micromouse-main-board/MicromouseV0.0.3.brd (EAGLE design)
At the start: 86 x 74 mm, 54 parts, among them U1 SN74HC151DR, U2 DRV8848PWPR, U3 ACS712ELCTR-20A-T

Commit message: Added debug header
Parts:
- added J1: (no value), SparkFun-Connectors:1X04
Connections:
- net 3V3: now also J1.4
- net GND: now also J1.1
- net SWCLK: now also J1.2
- net SWDIO: now also J1.3
Changed lines of the file:
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@@
 <attribute name="SPICEPREFIX" value="R" x="-124.587" y="-254.127" size="1.778" layer="27" display="off"/>
+</element>
+<element name="J1" library="SparkFun-Connectors" library_urn="urn:adsk.eagle:library:513" package="1X04" package3d_urn="urn:adsk.eagle:package:38085/1" value="" x="-124.841" y="-259.588">
+<attribute name="PROD_ID" value="CONN-09696" x="-124.841" y="-259.588" size="1.778" layer="27" display="off"/>
 </element>
 </elements>
@@
 <contactref element="U3" pad="5"/>
 <contactref element="CR1" pad="63"/>
-<wire x1="54.2172" y1="69.1642" x2="54.2172" y2="71.1962" width="0" layer="19" extent="1-1"/>
-<wire x1="54.879" y1="63.0326" x2="54.2172" y2="69.1642" width="0" layer="19" extent="1-1"/>
-<wire x1="55.2662" y1="61.3664" x2="54.879" y2="63.0326" width="0" layer="19" extent="1-1"/>
-<wire x1="45.27" y1="57.375" x2="55.2662" y2="61.3664" width="0" layer="19" extent="1-1"/>
-<wire x1="53.9254" y1="42.7609" x2="45.27" y2="57.375" width="0" layer="19" extent="1-1"/>
-<wire x1="51.5493" y1="35.3848" x2="53.9254" y2="42.7609" width="0" layer="19" extent="1-1"/>
-<wire x1="53.9254" y1="31.5087" x2="51.5493" y2="35.3848" width="0" layer="19" extent="1-1"/>
+<contactref element="J1" pad="1"/>
+<wire x1="-123.637" y1="-254.127" x2="-124.841" y2="-259.588" width="0" layer="19" extent="1-1"/>
+<wire x1="-124.245" y1="-248.539" x2="-123.637" y2="-254.127" width="0" layer="19" extent="1-1"/>
+<wire x1="-124.245" y1="-244.983" x2="-124.245" y2="-248.539" width="0" layer="19" extent="1-1"/>
+<wire x1="-124.245" y1="-241.427" x2="-124.245" y2="-244.983" width="0" layer="19" extent="1-1"/>
+<wire x1="-124.245" y1="-237.871" x2="-124.245" y2="-241.427" width="0" layer="19" extent="1-1"/>
+<wire x1="-124.245" y1="-234.315" x2="-124.245" y2="-237.871" width="0" layer="19" extent="1-1"/>
+<wire x1="-124.245" y1="-230.759" x2="-124.245" y2="-234.315" width="0" layer="19" extent="1-1"/>
+<wire x1="-124.245" y1="-227.203" x2="-124.245" y2="-230.759" width="0" layer="19" extent="1-1"/>
+<wire x1="-124.245" y1="-223.647" x2="-124.245" y2="-227.203" width="0" layer="19" extent="1-1"/>
+<wire x1="-120.0912" y1="-216.535" x2="-124.245" y2="-223.647" width="0" layer="19" extent="1-1"/>
+<wire x1="-106.35" y1="-215.829" x2="-120.0912" y2="-216.535" width="0" layer="19" extent="1-1"/>
+<wire x1="-101.3206" y1="-216.789" x2="-106.35" y2="-215.829" width="0" layer="19" extent="1-1"/>
+<wire x1="26.73" y1="16.625" x2="-101.3206" y2="-216.789" width="0" layer="19" extent="1-1"/>
+<wire x1="53.0234" y1="13.2588" x2="26.73" y2="16.625" width="0" layer="19" extent="1-1"/>
+<wire x1="53.0202" y1="11.364" x2="53.0234" y2="13.2588" width="0" layer="19" extent="1-1"/>
+<wire x1="54.0902" y1="5.1816" x2="53.0202" y2="11.364" width="0" layer="19" extent="1-1"/>
+<wire x1="54.0902" y1="3.1496" x2="54.0902" y2="5.1816" width="0" layer="19" extent="1-1"/>
+<wire x1="53.9254" y1="31.5087" x2="53.0234" y2="13.2588" width="0" layer="19" extent="1-1"/>
+<wire x1="51.5493" y1="35.3848" x2="53.9254" y2="31.5087" width="0" layer="19" extent="1-1"/>
 <wire x1="60.4254" y1="31.5087" x2="53.9254" y2="31.5087" width="0" layer="19" extent="1-1"/>
-<wire x1="62.8015" y1="40.3848" x2="53.9254" y2="42.7609" width="0" layer="19" extent="1-1"/>
+<wire x1="53.9254" y1="42.7609" x2="51.5493" y2="35.3848" width="0" layer="19" extent="1-1"/>
+<wire x1="62.8015" y1="40.3848" x2="60.4254" y2="31.5087" width="0" layer="19" extent="1-1"/>
 <wire x1="68.4784" y1="23.1784" x2="60.4254" y2="31.5087" width="0" layer="19" extent="1-1"/>
 <wire x1="69.9668" y1="23.5816" x2="68.4784" y2="23.1784" width="0" layer="19" extent="1-1"/>
@@
 <wire x1="74.7522" y1="48.1974" x2="76.4286" y2="36.1832" width="0" layer="19" extent="1-1"/>
 <wire x1="72.7202" y1="48.1974" x2="74.7522" y2="48.1974" width="0" layer="19" extent="1-1"/>
-<wire x1="53.0234" y1="13.2588" x2="53.9254" y2="31.5087" width="0" layer="19" extent="1-1"/>
-<wire x1="53.0202" y1="11.364" x2="53.0234" y2="13.2588" width="0" layer="19" extent="1-1"/>
-<wire x1="54.0902" y1="5.1816" x2="53.0202" y2="11.364" width="0" layer="19" extent="1-1"/>
-<wire x1="54.0902" y1="3.1496" x2="54.0902" y2="5.1816" width="0" layer="19" extent="1-1"/>
-<wire x1="26.73" y1="16.625" x2="53.0234" y2="13.2588" width="0" layer="19" extent="1-1"/>
-<wire x1="-101.3206" y1="-216.789" x2="26.73" y2="16.625" width="0" layer="19" extent="1-1"/>
-<wire x1="-106.35" y1="-215.829" x2="-101.3206" y2="-216.789" width="0" layer="19" extent="1-1"/>
-<wire x1="-120.0912" y1="-216.535" x2="-106.35" y2="-215.829" width="0" layer="19" extent="1-1"/>
-<wire x1="-124.245" y1="-223.647" x2="-120.0912" y2="-216.535" width="0" layer="19" extent="1-1"/>
-<wire x1="-124.245" y1="-227.203" x2="-124.245" y2="-223.647" width="0" layer="19" extent="1-1"/>
-<wire x1="-124.245" y1="-230.759" x2="-124.245" y2="-227.203" width="0" layer="19" extent="1-1"/>
-<wire x1="-124.245" y1="-234.315" x2="-124.245" y2="-230.759" width="0" layer="19" extent="1-1"/>
-<wire x1="-124.245" y1="-237.871" x2="-124.245" y2="-234.315" width="0" layer="19" extent="1-1"/>
-<wire x1="-124.245" y1="-241.427" x2="-124.245" y2="-237.871" width="0" layer="19" extent="1-1"/>
-<wire x1="-124.245" y1="-244.983" x2="-124.245" y2="-241.427" width="0" layer="19" extent="1-1"/>
-<wire x1="-124.245" y1="-248.539" x2="-124.245" y2="-244.983" width="0" layer="19" extent="1-1"/>
-<wire x1="-123.637" y1="-254.127" x2="-124.245" y2="-248.539" width="0" layer="19" extent="1-1"/>
+<wire x1="45.27" y1="57.375" x2="53.9254" y2="42.7609" width="0" layer="19" extent="1-1"/>
+<wire x1="55.2662" y1="61.3664" x2="45.27" y2="57.375" width="0" layer="19" extent="1-1"/>
+<wire x1="54.879" y1="63.0326" x2="55.2662" y2="61.3664" width="0" layer="19" extent="1-1"/>
+<wire x1="54.2172" y1="69.1642" x2="54.879" y2="63.0326" width="0" layer="19" extent="1-1"/>
+<wire x1="54.2172" y1="71.1962" x2="54.2172" y2="69.1642" width="0" layer="19" extent="1-1"/>
 </signal>
 <signal name="5V">
@@
 <signal name="SWCLK">
 <contactref element="CR1" pad="49"/>
+<contactref element="J1" pad="2"/>
+<wire x1="60.9254" y1="42.7609" x2="-122.301" y2="-259.588" width="0" layer="19" extent="1-1"/>
 </signal>
 <signal name="SWDIO">
 <contactref element="CR1" pad="46"/>
+<contactref element="J1" pad="3"/>
+<wire x1="62.8015" y1="39.8848" x2="-119.761" y2="-259.588" width="0" layer="19" extent="1-1"/>
 </signal>
 <signal name="NRST">
@@
 <contactref element="U1" pad="16"/>
 <contactref element="C3" pad="1"/>
+<contactref element="J1" pad="4"/>
+<wire x1="-125.945" y1="-248.539" x2="-117.221" y2="-259.588" width="0" layer="19" extent="1-1"/>
 <wire x1="-125.945" y1="-244.983" x2="-125.945" y2="-248.539" width="0" layer="19" extent="1-1"/>
 <wire x1="-125.945" y1="-234.315" x2="-125.945" y2="-244.983" width="0" layer="19" extent="1-1"/>

Commit message: added software repo, schematic not complete
Parts:
- moved J1 342.1 mm to (61.5, 27.3), turned to 90 degrees
- moved R1 334.6 mm to (56.0, 27.6), turned to 90 degrees
- moved C8 326.7 mm to (50.4, 27.1), turned to 90 degrees
- moved C7 321.8 mm to (46.9, 27.1), turned to 90 degrees
- moved C6 316.9 mm to (43.3, 27.1), turned to 90 degrees
- moved C5 312.0 mm to (39.8, 27.1), turned to 90 degrees
- moved C4 307.1 mm to (36.2, 27.1), turned to 90 degrees
- moved C3 302.2 mm to (32.6, 27.1), turned to 90 degrees
- moved C2 297.3 mm to (29.1, 27.1), turned to 90 degrees
- moved U1 295.8 mm to (18.7, 55.6), turned to 90 degrees
- moved C1 292.5 mm to (25.5, 27.1), turned to 90 degrees
- moved U2 288.6 mm to (18.0, 42.9), turned to 90 degrees
- moved U3 281.0 mm to (16.5, 29.6), turned to 90 degrees
