File: micromouse-main-board/MicromouseV0.0.6.brd (EAGLE design)
At the start: 86 x 75 mm, 89 parts, among them Q1 2.5A/30V, U1 SN74HC151DR, U2 DRV8848PWPR, U3 ACS712ELCTR-20A-T, U4 AP2112K-3.3V, U5 MCP73831

Commit message: update
Parts:
- added C2: 10uF, rcl:C0603
- added D4: (no value), diode:SMB
- added R10: 1k, rcl:M0805
- C1, C12, C13: value (none) -> 1uF
Connections:
- net (USART1)_RX: now also J2.2
- net (USART1)_TX: now also J2.3
- net ADC_IN: now also C2.1, R10.1
- net GND: now also C2.2, D4.A
- net N$2: now also D4.C, R10.2
Changed lines of the file:
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@@
 <?xml version="1.0" encoding="utf-8"?>
 <!DOCTYPE eagle SYSTEM "eagle.dtd">
-<eagle version="9.4.2">
+<eagle version="9.1.0">
 <drawing>
 <settings>
-<setting alwaysvectorfont="yes"/>
+<setting alwaysvectorfont="no"/>
 <setting verticaltext="up"/>
 </settings>
@@
 <attribute name="VALUE" x="7.62" y="63.627" size="1.778" layer="27" ratio="10" rot="R180"/>
 </element>
-<element name="C12" library="MicromouseV0.0.4" library_urn="urn:adsk.eagle:library:12230880" package="0603-CAP" package3d_urn="urn:adsk.eagle:package:12230963/1" value="" x="50.038" y="67.056" smashed="yes">
+<element name="C12" library="MicromouseV0.0.4" library_urn="urn:adsk.eagle:library:12230880" package="0603-CAP" package3d_urn="urn:adsk.eagle:package:12230963/1" value="1uF" x="50.038" y="67.056" smashed="yes">
 <attribute name="NAME" x="49.149" y="67.818" size="0.4064" layer="25" font="vector"/>
 <attribute name="VALUE" x="49.022" y="65.913" size="0.4064" layer="27" font="vector"/>
 </element>
-<element name="C13" library="MicromouseV0.0.4" library_urn="urn:adsk.eagle:library:12230880" package="0603-CAP" package3d_urn="urn:adsk.eagle:package:12230963/1" value="" x="50.038" y="64.516" smashed="yes">
+<element name="C13" library="MicromouseV0.0.4" library_urn="urn:adsk.eagle:library:12230880" package="0603-CAP" package3d_urn="urn:adsk.eagle:package:12230963/1" value="1uF" x="50.038" y="64.516" smashed="yes">
 <attribute name="NAME" x="49.149" y="65.278" size="0.4064" layer="25" font="vector"/>
 <attribute name="VALUE" x="49.022" y="63.373" size="0.4064" layer="27" font="vector"/>
 </element>
-<element name="C1" library="MicromouseV0.0.4" library_urn="urn:adsk.eagle:library:12230880" package="0603-CAP" package3d_urn="urn:adsk.eagle:package:12230963/1" value="" x="50.038" y="61.976" smashed="yes">
+<element name="C1" library="MicromouseV0.0.4" library_urn="urn:adsk.eagle:library:12230880" package="0603-CAP" package3d_urn="urn:adsk.eagle:package:12230963/1" value="1uF" x="50.038" y="61.976" smashed="yes">
 <attribute name="NAME" x="49.149" y="62.738" size="0.4064" layer="25" font="vector"/>
 <attribute name="VALUE" x="49.022" y="60.833" size="0.4064" layer="27" font="vector"/>
@@
 <attribute name="PROD_ID" value="CONN-09696" x="65.024" y="25.273" size="1.778" layer="27" rot="R90" display="off"/>
 <attribute name="VALUE" x="67.056" y="24.003" size="0.6096" layer="27" font="vector" ratio="20" rot="R90"/>
+</element>
+<element name="D4" library="diode" library_urn="urn:adsk.eagle:library:210" package="SMB" package3d_urn="urn:adsk.eagle:package:43404/2" value="" x="-88.773" y="-225.171"/>
+<element name="R10" library="rcl" library_urn="urn:adsk.eagle:library:334" package="M0805" package3d_urn="urn:adsk.eagle:package:23556/2" value="1k" x="-90.297" y="-230.251">
+<attribute name="SPICEPREFIX" value="R" x="-90.297" y="-230.251" size="1.778" layer="27" display="off"/>
+</element>
+<element name="C2" library="rcl" library_urn="urn:adsk.eagle:library:334" package="C0603" package3d_urn="urn:adsk.eagle:package:23616/2" value="10uF" x="-90.805" y="-235.839">
+<attribute name="SPICEPREFIX" value="C" x="-90.805" y="-235.839" size="1.778" layer="27" display="off"/>
 </element>
 </elements>
@@
 <contactref element="C18" pad="1"/>
 <contactref element="J2" pad="1"/>
+<contactref element="D4" pad="A"/>
+<contactref element="C2" pad="2"/>
 <wire x1="72.7202" y1="48.1974" x2="74.7522" y2="48.1974" width="0" layer="19" extent="1-1"/>
 <wire x1="63.4365" y1="48.5128" x2="72.7202" y2="48.1974" width="0" layer="19" extent="1-1"/>
@@
 <wire x1="55.9952" y1="58.2422" x2="55.0122" y2="56.2864" width="0" layer="19" extent="1-1"/>
 <wire x1="54.879" y1="59.2226" x2="55.9952" y2="58.2422" width="0" layer="19" extent="1-1"/>
-<wire x1="49.6452" y1="61.7982" x2="54.879" y2="59.2226" width="0" layer="19" extent="1-1"/>
-<wire x1="52.1843" y1="43.5128" x2="54.5604" y2="50.8889" width="0" layer="19" extent="1-1"/>
+<wire x1="50.888" y1="59.436" x2="54.879" y2="59.2226" width="0" layer="19" extent="1-1"/>
+<wire x1="50.888" y1="61.976" x2="50.888" y2="59.436" width="0" layer="19" extent="1-1"/>
+<wire x1="49.6452" y1="61.7982" x2="50.888" y2="61.976" width="0" layer="19" extent="1-1"/>
+<wire x1="50.888" y1="64.516" x2="50.888" y2="61.976" width="0" layer="19" extent="1-1"/>
+<wire x1="50.888" y1="67.056" x2="50.888" y2="64.516" width="0" layer="19" extent="1-1"/>
+<wire x1="50.888" y1="56.896" x2="50.888" y2="59.436" width="0" layer="19" extent="1-1"/>
+<wire x1="47.586" y1="51.816" x2="50.888" y2="56.896" width="0" layer="19" extent="1-1"/>
+<wire x1="47.586" y1="48.768" x2="47.586" y2="51.816" width="0" layer="19" extent="1-1"/>
+<wire x1="42.788" y1="49.022" x2="47.586" y2="48.768" width="0" layer="19" extent="1-1"/>
+<wire x1="39.74" y1="49.022" x2="42.788" y2="49.022" width="0" layer="19" extent="1-1"/>
+<wire x1="41.49" y1="45.72" x2="42.788" y2="49.022" width="0" layer="19" extent="1-1"/>
+<wire x1="39.79" y1="43.18" x2="41.49" y2="45.72" width="0" layer="19" extent="1-1"/>
+<wire x1="52.1843" y1="43.5128" x2="47.586" y2="48.768" width="0" layer="19" extent="1-1"/>
 <wire x1="54.5604" y1="39.6367" x2="52.1843" y2="43.5128" width="0" layer="19" extent="1-1"/>
 <wire x1="61.0604" y1="39.6367" x2="54.5604" y2="39.6367" width="0" layer="19" extent="1-1"/>
-<wire x1="41.333" y1="58.01" x2="49.6452" y2="61.7982" width="0" layer="19" extent="1-1"/>
+<wire x1="41.333" y1="58.01" x2="47.586" y2="51.816" width="0" layer="19" extent="1-1"/>
 <wire x1="56.007" y1="28.509" x2="54.5604" y2="39.6367" width="0" layer="19" extent="1-1"/>
 <wire x1="50.419" y1="27.901" x2="56.007" y2="28.509" width="0" layer="19" extent="1-1"/>
 <wire x1="46.863" y1="27.901" x2="50.419" y2="27.901" width="0" layer="19" extent="1-1"/>
 <wire x1="62.357" y1="25.273" x2="56.007" y2="28.509" width="0" layer="19" extent="1-1"/>
-<wire x1="68.4784" y1="23.1784" x2="62.357" y2="25.273" width="0" layer="19" extent="1-1"/>
+<wire x1="65.024" y1="25.273" x2="62.357" y2="25.273" width="0" layer="19" extent="1-1"/>
+<wire x1="68.4784" y1="23.1784" x2="65.024" y2="25.273" width="0" layer="19" extent="1-1"/>
 <wire x1="69.9668" y1="23.5816" x2="68.4784" y2="23.1784" width="0" layer="19" extent="1-1"/>
 <wire x1="71.6534" y1="28.5632" x2="69.9668" y2="23.5816" width="0" layer="19" extent="1-1"/>
@@
 <wire x1="53.0202" y1="11.364" x2="53.0234" y2="13.2588" width="0" layer="19" extent="1-1"/>
 <wire x1="44.6922" y1="14.3256" x2="51.0422" y2="19.1516" width="0" layer="19" extent="1-1"/>
-<wire x1="35.941" y1="32.219" x2="46.863" y2="27.901" width="0" layer="19" extent="1-1"/>
+<wire x1="35.941" y1="32.219" x2="39.79" y2="43.18" width="0" layer="19" extent="1-1"/>
 <wire x1="29.591" y1="32.473" x2="35.941" y2="32.219" width="0" layer="19" extent="1-1"/>
 <wire x1="24.511" y1="41.9354" x2="29.591" y2="32.473" width="0" layer="19" extent="1-1"/>
@@
 <wire x1="8.908" y1="5.296" x2="13.462" y2="16.2861" width="0" layer="19" extent="1-1"/>
 <wire x1="4.808" y1="5.296" x2="8.908" y2="5.296" width="0" layer="19" extent="1-1"/>
-<wire x1="50.888" y1="67.056" x2="4.808" y2="5.296" width="0" layer="19" extent="1-1"/>
-<wire x1="50.888" y1="64.516" x2="50.888" y2="67.056" width="0" layer="19" extent="1-1"/>
-<wire x1="50.888" y1="61.976" x2="50.888" y2="64.516" width="0" layer="19" extent="1-1"/>
-<wire x1="50.888" y1="59.436" x2="50.888" y2="61.976" width="0" layer="19" extent="1-1"/>
-<wire x1="50.888" y1="56.896" x2="50.888" y2="59.436" width="0" layer="19" extent="1-1"/>
-<wire x1="47.586" y1="51.816" x2="50.888" y2="56.896" width="0" layer="19" extent="1-1"/>
-<wire x1="47.586" y1="48.768" x2="47.586" y2="51.816" width="0" layer="19" extent="1-1"/>
-<wire x1="42.788" y1="49.022" x2="47.586" y2="48.768" width="0" layer="19" extent="1-1"/>
-<wire x1="39.74" y1="49.022" x2="42.788" y2="49.022" width="0" layer="19" extent="1-1"/>
-<wire x1="41.49" y1="45.72" x2="42.788" y2="49.022" width="0" layer="19" extent="1-1"/>
-<wire x1="39.79" y1="43.18" x2="41.49" y2="45.72" width="0" layer="19" extent="1-1"/>
-<wire x1="65.024" y1="25.273" x2="39.79" y2="43.18" width="0" layer="19" extent="1-1"/>
+<wire x1="-86.573" y1="-225.171" x2="4.808" y2="5.296" width="0" layer="19" extent="1-1"/>
+<wire x1="-89.955" y1="-235.839" x2="-86.573" y2="-225.171" width="0" layer="19" extent="1-1"/>
 </signal>
 <signal name="5V">
@@
 <signal name="ADC_IN">
 <contactref element="CR1" pad="11"/>
+<contactref element="R10" pad="1"/>
+<contactref element="C2" pad="1"/>
+<wire x1="-91.247" y1="-230.251" x2="52.1843" y2="44.0128" width="0" layer="19" extent="1-1"/>
+<wire x1="-91.655" y1="-235.839" x2="-91.247" y2="-230.251" width="0" layer="19" extent="1-1"/>
 </signal>
 <signal name="N$9">
@@
 <contactref element="C13" pad="1"/>
 <wire x1="9.271" y1="29.6672" x2="49.188" y2="64.516" width="0" layer="19" extent="1-1"/>
-</signal>
-<signal name="N$2">
-<contactref element="U1" pad="5"/>
 </signal>
 <signal name="N$3">
@@
 <signal name="(USART1)_RX">
 <contactref element="CR1" pad="42"/>
+<contactref element="J2" pad="2"/>
+<wire x1="65.024" y1="27.813" x2="63.4365" y2="46.0128" width="0" layer="19" extent="1-1"/>
 </signal>
 <signal name="(USART1)_TX">
 <contactref element="CR1" pad="43"/>
+<contactref element="J2" pad="3"/>
+<wire x1="65.024" y1="30.353" x2="63.4365" y2="46.5128" width="0" layer="19" extent="1-1"/>
+</signal>
+<signal name="N$2">
+<contactref element="U1" pad="5"/>
+<contactref element="D4" pad="C"/>
+<contactref element="R10" pad="2"/>
+<wire x1="-90.973" y1="-225.171" x2="-89.347" y2="-230.251" width="0" layer="19" extent="1-1"/>
+<wire x1="20.701" y1="41.9354" x2="-90.973" y2="-225.171" width="0" layer="19" extent="1-1"/>
 </signal>
 </signals>
