File: micromouse-main-board/MicromouseV0.0.6.sch (EAGLE design)
At the start: 89 parts, among them Q1 2.5A/30V, U1 SN74HC151DR, U2 DRV8848PWPR, U3 ACS712ELCTR-20A-T, U4 AP2112K-3.3V, U5 MCP73831

Commit message: update
Parts:
- added C2: 10uF, rcl:C-USC0603
- added D4: (no value), diode:ZENER-DIODESMB
- added R10: 1k, rcl:R-US_M0805
- C1, C12, C13: value (none) -> 1uF
Connections:
- net (USART1)_RX: now also J2.2
- net (USART1)_TX: now also J2.3
- net ADC_IN: now also C2.1, R10.1
- net GND: now also C2.2, D4.A
- net N$2: now also D4.C, R10.2
Other:
- note added: "NOTE: RC VALUES ARE NOT SET YET THESE ARE PLACEHOLDER VALUES"
Changed lines of the file:
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@@
 <?xml version="1.0" encoding="utf-8"?>
 <!DOCTYPE eagle SYSTEM "eagle.dtd">
-<eagle version="9.4.2">
+<eagle version="9.1.0">
 <drawing>
 <settings>
@@
 <setting verticaltext="up"/>
 </settings>
-<grid distance="0.01" unitdist="inch" unit="inch" style="lines" multiple="1" display="yes" altdistance="0.01" altunitdist="inch" altunit="inch"/>
+<grid distance="0.05" unitdist="inch" unit="inch" style="lines" multiple="1" display="no" altdistance="0.01" altunitdist="inch" altunit="inch"/>
 <layers>
 <layer number="1" name="Top" color="4" fill="1" visible="no" active="no"/>
@@
 <part name="V_BATT" library="SparkFun-Aesthetics" deviceset="V_BATT" device=""/>
 <part name="SUPPLY1" library="Corgi_V3.8.5" library_urn="urn:adsk.eagle:library:8483107" deviceset="VCC" device="" value="3.3V"/>
-<part name="C12" library="MicromouseV0.0.4" library_urn="urn:adsk.eagle:library:12230880" deviceset="CAP" device="0603-CAP" package3d_urn="urn:adsk.eagle:package:12230963/1"/>
-<part name="C13" library="MicromouseV0.0.4" library_urn="urn:adsk.eagle:library:12230880" deviceset="CAP" device="0603-CAP" package3d_urn="urn:adsk.eagle:package:12230963/1"/>
+<part name="C12" library="MicromouseV0.0.4" library_urn="urn:adsk.eagle:library:12230880" deviceset="CAP" device="0603-CAP" package3d_urn="urn:adsk.eagle:package:12230963/1" value="1uF"/>
+<part name="C13" library="MicromouseV0.0.4" library_urn="urn:adsk.eagle:library:12230880" deviceset="CAP" device="0603-CAP" package3d_urn="urn:adsk.eagle:package:12230963/1" value="1uF"/>
 <part name="SUPPLY5" library="Corgi_V3.8.5" library_urn="urn:adsk.eagle:library:8483107" deviceset="VCC" device=""/>
-<part name="C1" library="MicromouseV0.0.4" library_urn="urn:adsk.eagle:library:12230880" deviceset="CAP" device="0603-CAP" package3d_urn="urn:adsk.eagle:package:12230963/1"/>
+<part name="C1" library="MicromouseV0.0.4" library_urn="urn:adsk.eagle:library:12230880" deviceset="CAP" device="0603-CAP" package3d_urn="urn:adsk.eagle:package:12230963/1" value="1uF"/>
 <part name="GND5" library="supply1" library_urn="urn:adsk.eagle:library:371" deviceset="GND" device=""/>
 <part name="C5" library="MicromouseV0.0.4" library_urn="urn:adsk.eagle:library:12230880" deviceset="CAP" device="0603-CAP" package3d_urn="urn:adsk.eagle:package:12230963/1"/>
@@
 <part name="SUPPLY3" library="Corgi_V4.13.0" library_urn="urn:adsk.eagle:library:10157911" deviceset="VCC" device="" value="3.3V"/>
 <part name="J2" library="MicromouseV0.0.4" library_urn="urn:adsk.eagle:library:12230880" deviceset="CONN_04" device="" package3d_urn="urn:adsk.eagle:package:12230952/1"/>
+<part name="D4" library="diode" library_urn="urn:adsk.eagle:library:210" deviceset="ZENER-DIODE" device="SMB" package3d_urn="urn:adsk.eagle:package:43404/2"/>
+<part name="GND6" library="supply1" library_urn="urn:adsk.eagle:library:371" deviceset="GND" device=""/>
+<part name="R10" library="rcl" library_urn="urn:adsk.eagle:library:334" deviceset="R-US_" device="M0805" package3d_urn="urn:adsk.eagle:package:23556/2" value="1k"/>
+<part name="C2" library="rcl" library_urn="urn:adsk.eagle:library:334" deviceset="C-US" device="C0603" package3d_urn="urn:adsk.eagle:package:23616/2" value="10uF"/>
+<part name="GND44" library="supply1" library_urn="urn:adsk.eagle:library:371" deviceset="GND" device=""/>
 </parts>
 <sheets>
@@
 <wire x1="231.902" y1="136.144" x2="231.902" y2="257.556" width="0.1524" layer="97" style="longdash"/>
 <wire x1="231.902" y1="257.556" x2="403.352" y2="257.556" width="0.1524" layer="97" style="longdash"/>
+<text x="48.26" y="-22.86" size="1.778" layer="94">NOTE: RC VALUES ARE NOT SET YET THESE ARE PLACEHOLDER VALUES</text>
 </plain>
 <instances>
@@
 <attribute name="VALUE" x="192.532" y="-29.972" size="1.778" layer="96" font="vector"/>
 <attribute name="NAME" x="192.532" y="-14.478" size="1.778" layer="95" font="vector"/>
+</instance>
+<instance part="D4" gate="G$1" x="78.74" y="-38.1" rot="R90"/>
+<instance part="GND6" gate="1" x="78.716946875" y="-46.674503125" smashed="yes">
+<attribute name="VALUE" x="76.176946875" y="-49.214503125" size="1.778" layer="96"/>
+</instance>
+<instance part="R10" gate="G$1" x="93.98" y="-34.29" smashed="yes" rot="R180">
+<attribute name="NAME" x="97.79" y="-35.7886" size="1.778" layer="95" rot="R180"/>
+<attribute name="VALUE" x="97.79" y="-30.988" size="1.778" layer="96" rot="R180"/>
+</instance>
+<instance part="C2" gate="G$1" x="111.76" y="-38.1" smashed="yes">
+<attribute name="NAME" x="112.776" y="-37.465" size="1.778" layer="95"/>
+<attribute name="VALUE" x="112.776" y="-42.291" size="1.778" layer="96"/>
+</instance>
+<instance part="GND44" gate="1" x="111.736946875" y="-46.674503125" smashed="yes">
+<attribute name="VALUE" x="109.196946875" y="-49.214503125" size="1.778" layer="96"/>
 </instance>
 </instances>
@@
 <label x="203.2" y="-25.146" size="1.27" layer="95" xref="yes"/>
 </segment>
+<segment>
+<pinref part="GND6" gate="1" pin="GND"/>
+<pinref part="D4" gate="G$1" pin="A"/>
+<wire x1="78.716946875" y1="-44.134503125" x2="78.74" y2="-44.134503125" width="0.1524" layer="91"/>
+<wire x1="78.74" y1="-44.134503125" x2="78.74" y2="-40.64" width="0.1524" layer="91"/>
+</segment>
+<segment>
+<pinref part="GND44" gate="1" pin="GND"/>
+<pinref part="C2" gate="G$1" pin="2"/>
+<wire x1="111.736946875" y1="-44.134503125" x2="111.76" y2="-44.134503125" width="0.1524" layer="91"/>
+<wire x1="111.76" y1="-44.134503125" x2="111.76" y2="-43.18" width="0.1524" layer="91"/>
+</segment>
 </net>
 <net name="5V" class="0">
@@
 <pinref part="CR1" gate="A" pin="PC3"/>
 <wire x1="274.32" y1="-134.62" x2="271.272" y2="-134.874" width="0.1524" layer="91"/>
-<label x="264.922" y="-133.35" size="1.778" layer="95" rot="R180"/>
+<label x="271.272" y="-134.62" size="1.778" layer="95" rot="R180"/>
+</segment>
+<segment>
+<pinref part="R10" gate="G$1" pin="1"/>
+<pinref part="C2" gate="G$1" pin="1"/>
+<wire x1="99.06" y1="-34.29" x2="111.76" y2="-34.29" width="0.1524" layer="91"/>
+<wire x1="111.76" y1="-34.29" x2="111.76" y2="-35.56" width="0.1524" layer="91"/>
+<wire x1="111.76" y1="-34.29" x2="120.65" y2="-34.29" width="0.1524" layer="91"/>
+<junction x="111.76" y="-34.29"/>
+<label x="120.65" y="-34.29" size="1.778" layer="95"/>
 </segment>
 </net>
@@
 <wire x1="187.96" y1="-149.352" x2="187.96" y2="-149.606" width="0.1524" layer="91"/>
 <junction x="187.96" y="-149.352"/>
-</segment>
-</net>
-<net name="N$2" class="0">
-<segment>
-<pinref part="U1" gate="A" pin="Y"/>
-<wire x1="66.802" y1="-34.036" x2="71.882" y2="-34.036" width="0.1524" layer="91"/>
 </segment>
 </net>
@@
 <label x="476.25" y="-114.3" size="1.27" layer="95" xref="yes"/>
 </segment>
+<segment>
+<pinref part="J2" gate="G$1" pin="2"/>
+<wire x1="202.692" y1="-22.606" x2="202.692" y2="-22.86" width="0.1524" layer="91"/>
+<wire x1="202.692" y1="-22.86" x2="205.74" y2="-22.86" width="0.1524" layer="91"/>
+<label x="205.74" y="-22.86" size="1.778" layer="95"/>
+</segment>
 </net>
 <net name="(USART1)_TX" class="0">
@@
 <label x="476.25" y="-109.22" size="1.27" layer="95" xref="yes"/>
 </segment>
-</net>
+<segment>
+<pinref part="J2" gate="G$1" pin="3"/>
+<wire x1="202.692" y1="-20.066" x2="205.74" y2="-20.066" width="0.1524" layer="91"/>
+<wire x1="205.74" y1="-20.066" x2="205.74" y2="-20.32" width="0.1524" layer="91"/>
+<label x="205.74" y="-20.32" size="1.778" layer="95"/>
+</segment>
+</net>
+<net name="N$2" class="0">
+<segment>
+<pinref part="U1" gate="A" pin="Y"/>
+<pinref part="D4" gate="G$1" pin="C"/>
+<wire x1="66.802" y1="-34.036" x2="78.74" y2="-34.036" width="0.1524" layer="91"/>
+<wire x1="78.74" y1="-34.036" x2="78.74" y2="-34.29" width="0.1524" layer="91"/>
+<pinref part="R10" gate="G$1" pin="2"/>
+<wire x1="78.74" y1="-34.29" x2="78.74" y2="-35.56" width="0.1524" layer="91"/>
+<wire x1="88.9" y1="-34.29" x2="78.74" y2="-34.29" width="0.1524" layer="91"/>
+<junction x="78.74" y="-34.29"/>
+</segment>
+</net>

Commit message: update
Other:
- note added: "NOTE: RC VALUES ARE NOT SET YET THESE ARE PLACEHOLDER VALUES. MIGHT ALSO NEED OP AMP AT END OF CIRCUIT"
- note removed: "NOTE: RC VALUES ARE NOT SET YET THESE ARE PLACEHOLDER VALUES"
Changed lines of the file:
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@@
 <wire x1="231.902" y1="136.144" x2="231.902" y2="257.556" width="0.1524" layer="97" style="longdash"/>
 <wire x1="231.902" y1="257.556" x2="403.352" y2="257.556" width="0.1524" layer="97" style="longdash"/>
-<text x="48.26" y="-22.86" size="1.778" layer="94">NOTE: RC VALUES ARE NOT SET YET THESE ARE PLACEHOLDER VALUES</text>
+<text x="-7.62" y="-20.32" size="1.778" layer="94">NOTE: RC VALUES ARE NOT SET YET THESE ARE PLACEHOLDER VALUES. MIGHT ALSO NEED OP AMP AT END OF CIRCUIT</text>
 </plain>
 <instances>
