File: micromouse-main-board/micromouse-edu-boardV0.0.1.brd (EAGLE design)
At the start: 93.9 x 75 mm, 113 parts, among them IC1 LM321MFX, J3 HTSS-103-XX-XX-D, J5 HTSS-103-XX-XX-D, J6 HTSS-102-XX-XX-D, J7 HTSS-102-XX-XX-D, U1 SN74HC151DR, U2 DRV8848PWPR, U3 ACS712ELCTR-20A-T, U6 MPU-6000, X1 RASPI_GPIO_B+#_PIN

Commit message: added updated bom and changed some board components,these few traces will still need to be routed
Parts:
- added C10: 10nF, MicromouseV0.0.4:0603-CAP
- added C_5V3: 0.1uF, SparkFun:0603-CAP
- C1: value 1.1uF -> 1.0uF
- C13: value 0.01uF -> 1nF
- C_5V2: device SparkFun:1210 -> SparkFun:0603-CAP
- C_BAT2: value 47uF -> 0.1uF; device SparkFun:1210 -> SparkFun-Capacitors:0603-CAP
- R_VM1: value 75k -> 100k
- R_VM2: value 25k -> 33k
- moved C_5V2 1238.3 mm to (-1203.4, -225.6)
- moved C_BAT2 1234.5 mm to (-1203.4, -228.6), turned to 0 degrees
- renumbered LEFT_FRONT_EMITTER to E1, REC_LF to REC_1, U$11 to E3, U$13 to E4, U$17 to E2, U$18 to E5, U$19 to E6, U$20 to REC_5, U$21 to REC_6, U$7 to REC_2, U$8 to REC_3, U$9 to REC_4
Connections:
- net 3.3V: now also C10.2
- net GND: now also C10.1
Routing:
- net 5V: track 406.2 -> 403.5 mm
- net GND: track 336.5 -> 334.2 mm
- net V_BATT: track 47.5 -> 45.6 mm
