File: micromouse-main-board/micromouse-edu-boardV0.0.1.sch (EAGLE design)
At the start: 113 parts, among them IC1 LM321MFX, J3 HTSS-103-XX-XX-D, J5 HTSS-103-XX-XX-D, J6 HTSS-102-XX-XX-D, J7 HTSS-102-XX-XX-D, U1 SN74HC151DR, U2 DRV8848PWPR, U3 ACS712ELCTR-20A-T, U6 MPU-6000, X1 RASPI_GPIO_B+#_PIN

Commit message: added updated bom and changed some board components,these few traces will still need to be routed
Parts:
- added C10: 10nF, MicromouseV0.0.4:CAP0603-CAP
- added C_5V3: 0.1uF, SparkFun:CAP0603-CAP
- C1: value 1.1uF -> 1.0uF
- C13: value 0.01uF -> 1nF
- C_5V2: device SparkFun:CAP1210 -> SparkFun:CAP0603-CAP
- C_BAT2: value 47uF -> 0.1uF; device SparkFun:CAP1210 -> SparkFun-Capacitors:CAP0603-CAP
- R_VM1: value 75k -> 100k
- R_VM2: value 25k -> 33k
- renumbered LEFT_FRONT_EMITTER to E1, REC_LF to REC_1, U$11 to E3, U$13 to E4, U$17 to E2, U$18 to E5, U$19 to E6, U$20 to REC_5, U$21 to REC_6, U$7 to REC_2, U$8 to REC_3, U$9 to REC_4
Connections:
- net 3.3V: now also C10.2
- net GND: now also C10.1
