File: micromouse-main-board/micromouse-edu-finalV2.0.0.sch (EAGLE design)
At the start: 113 parts, among them IC1 LM321MFX, J3 HTSS-103-XX-XX-D, J5 HTSS-103-XX-XX-D, J6 HTSS-102-XX-XX-D, J7 HTSS-102-XX-XX-D, U1 SN74HC151DR, U2 DRV8848PWPR, U3 ACS712ELCTR-20A-T, U6 MPU-6000, X1 RASPI_GPIO_B+#_PIN

Commit message: value update to reflect bom
Parts:
- removed J7: HTSS-102-XX-XX-D, HTSS-102-01-G-D:HTSS-102-XX-XX-D
- C4: value 0.1uF -> 0.01uF
- R_VM2: value 25k -> 33k
Connections:
- removed net GPIO_BREAKOUT_1: J7.2, X1.GPIO27
- removed net GPIO_BREAKOUT_2: J7.4, X1.GPIO22
- removed net PWM_BREAKOUT_1: J7.1, X1.GPIO18
- removed net PWM_BREAKOUT_2: J7.3, X1.GPIO24
Other:
- note added: "33k"
- note removed: "still under construction"
