File: micromouse-main-board/micromouse-revB/micromouse_board_revB_V0.0.3.brd (EAGLE design)
At the start: 93.9 x 75 mm, 116 parts, among them IC1 LM321MFX, J3 HTSS-103-XX-XX-D, J5 HTSS-103-XX-XX-D, J6 HTSS-102-XX-XX-D, U1 SN74HC151DR, U2 DRV8848PWPR, U3 ACS712ELCTR-20A-T, U6 MPU-6000, X1 RASPI_GPIO_B+#_PIN

Commit message: power reg. added placement done
Parts:
- removed C12: 0.1 uF, micromouse-board-added-piconnector:0603-CAP
- removed C13: 0.01uF, micromouse-board-added-piconnector:0603-CAP
- removed C15: 10uF, micromouse-board-added-piconnector:0603-CAP
- removed C16, C9: 2.2uF, micromouse-board-added-piconnector:0603-CAP
- removed C20: 1000pF, micromouse-board-added-piconnector:0603-CAP
- removed C3: 1.4 uF, micromouse-board-added-piconnector:0603-CAP
- removed C5, C6: 0.1uF, micromouse-board-added-piconnector:0603-CAP
- removed D1: (no value), diode:SOT23
- removed IC1: LM321MFX, micromouse-board-added-piconnector:SOT23-5
- removed J2: (no value), micromouse-board-added-piconnector:1X04
- removed J3, J5: HTSS-103-XX-XX-D, micromouse-board-added-piconnector:HTSS-103-XX-XX-D
- removed J6: HTSS-102-XX-XX-D, micromouse-board-added-piconnector:HTSS-102-XX-XX-D
- removed JP1, JP3: (no value), micromouse-board-added-piconnector:MOLEX-1X2
- removed R3: 1k, rcl:R0805
- removed R6: 10k, rcl:M0805
- removed R8, R9: 500m, micromouse-board-added-piconnector:0805
- removed R_VM6: 3.3k, micromouse-board-added-piconnector:0603-RES
- removed R_VM7: 1k, micromouse-board-added-piconnector:0603-RES
- removed S1: RESET, micromouse-board-added-piconnector:TACTILE_SWITCH_SMD_4.6X2.8MM
- removed S3: (no value), micromouse-board-added-piconnector:SWITCH-SPDT
- removed U3: ACS712ELCTR-20A-T, micromouse-board-added-piconnector:SOIC127P600X175-8N
- added B1: (no value), SparkFun-Retired:TACTILE-SWITCH-SMD
- added C_1, C_3.3V4, C_D, C_NR1, C_NR2, C_NR3: 0.1uF, micromouse-board-added-piconnector:0603-CAP
- added C_3.3V3, C_3.3V7, C_3.3V8, C_3.3V9, C_D1: 10uF, micromouse-board-added-piconnector:0603-CAP
- added C_3.3V5, C_3.3V6, C_D2: 22uF, micromouse-board-added-piconnector:0603-CAP
- added C_NRST: 0.1uF, SparkFun:0603-CAP
- added L2: 10uH, micromouse-board-added-piconnector:1007
- added LED_PWR1: green, micromouse-board-added-piconnector:LED-1206
- added R_B1, R_B2: 47k, SparkFun-Passives:0603-RES
- added R_B3, R_B4: 1k, SparkFun-Passives:0603-RES
- added R_PWR1: 1k, micromouse-board-added-piconnector:0603-RES
- added R_VM3: 500m, micromouse-board-added-piconnector:0603-RES
- added U$10, U$5, U$6: 6P_HEADER, micro-motor:6P_HEADER
- added U$14, U$15: SPARKFUN-SPDT, micro-motor:SPDT
- added U$16, U$22: SPLITTER, splitter:SPLITTER
- added U$23: TPS73633(SOT-23), micromouse-board-added-piconnector:TPS73633(SOT-23)
- L1: value 10uH -> 4.7uH
- R1: value 1k -> 68k; device rcl:M0805 -> micromouse-board-added-piconnector:0603-RES
- R2: device micromouse-board-added-piconnector:0805 -> micromouse-board-added-piconnector:0603-RES
- R4, R5: value 10k -> 4.6k
- R_PWR: value 1k -> 500 Ohms
- R_VM2: value 25k -> 40k
- R_VM4: value 100k -> 500m
- R_VM5: value 100k -> 10k
- U$12: value MY_MM_MOTOR_MOUNT -> 6P_HEADER; device micromouse-board-added-piconnector:MY_MM_MOTOR_MOUNT -> micro-motor:6P_HEADER
- U1: value SN74HC151DR -> TPS561201DDCT; device micromouse-board-added-piconnector:SOIC127P600X175-16N -> micromouse-board-added-piconnector:DDC6
- moved R1 328.8 mm to (-90.7, -236.2), turned to 0 degrees
- moved U1 306.3 mm to (-88.4, -232.9)
- moved L1 302.3 mm to (-93.7, -241.3), turned to 0 degrees
- moved R2 301.7 mm to (-90.7, -239.3), turned to 0 degrees
- moved U6 66.3 mm to (48.6, 63.5)
- moved R4 53.7 mm to (55.3, 3.30)
- moved U$4 49.1 mm to (44.6, 12.6)
- moved R5 39.2 mm to (28.5, 34.4)
- moved U$3 38.8 mm to (43.8, 53.3)
- moved LED_PWR 38.0 mm to (-6.30, 14.2), turned to 180 degrees
- moved R_PWR 36.2 mm to (-1.60, 13.9)
- moved C_GY_VDD 30.3 mm to (33.3, 34.0), turned to 0 degrees
- moved C_BAT2 29.8 mm to (28.6, 49.1)
- moved NMOS2 29.0 mm to (55.0, 9.33), turned to 90 degrees
- moved C_3.3V2 28.4 mm to (36.5, 54.0)
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Connections:
- net (USART1)_RX renamed USART1_RX
- net (USART1)_TX renamed USART1_TX
- removed net I_SENSE: U1.13
- removed net LEFT_MOTOR_H: J5.2, JP1.1, U$12.L_MOTOR_A, U2.2
- removed net LEFT_MOTOR_L: J5.1, JP1.2, U$12.L_MOTOR_B, U2.4
- removed net MUX_EN: CR1.44, U1.7
- removed net N$20: R8.2, U2.6
- removed net N$21: IC1.1, R_VM4.2, R_VM5.1
- removed net N$24: R_VM7.2, U3.7
- removed net N$31: C20.2, IC1.3, R_VM6.1, R_VM7.1
- removed net NRST: C5.1, CR1.7, S1.3, S1.4
- removed net NSLEEP: U2.1
- removed net PWM_MOTOR_1: CR1.15, J6.1, U2.16
- removed net PWM_MOTOR_2: CR1.16, J6.2, U2.15
- removed net PWM_MOTOR_3: CR1.26, J6.3, U2.9
- removed net PWM_MOTOR_4: CR1.27, J6.4, U2.10
- removed net RIGHT_MOTOR_H: J3.2, JP3.1, U$12.R_MOTOR_A, U2.7
- removed net RIGHT_MOTOR_L: J3.1, JP3.2, U$12.R_MOTOR_B, U2.5
- removed net SEL_A: U1.11
- removed net SEL_B: U1.10
- removed net SEL_C: U1.9
- removed net SENSOR_DEBUG: C3.1, J2.4, R3.2
- new net 6V: C_3.3V5.1, C_3.3V6.1, L1.2, R1.2, U$10.3, U$12.3, U$5.3, U$6.3, U1.5
- new net BOOT0: CR1.60, U$14.P$2
- new net BOOT1: CR1.28, U$15.P$2
- new net BRIDGE_A_1: CR1.15, U2.16
- new net BRIDGE_A_2: CR1.16, U2.15
- new net BRIDGE_B_1: CR1.26, U2.9
- new net BRIDGE_B_2: CR1.27, U2.10
- new net M1_A: U$12.1, U$6.1, U2.2
- new net M1_B: U$12.2, U$6.2, U2.4
- new net M1_ENC_A: U$12.4, U$6.4
- new net M1_ENC_B: U$12.5, U$6.5
- new net M2_A: U$10.1, U$5.1, U2.7
- new net M2_B: U$10.2, U$5.2, U2.5
- new net M2_ENC_A: U$10.5, U$5.4
- new net M2_ENC_B: U$10.4, U$5.5
- new net MGND: C_D.2, C_D1.2, C_D2.2, R_VM3.2, R_VM4.2, U$10.6, U$12.6, U$16.2, U$5.6, U$6.6, U2.13
- new net N$10: C_D.1, C_D1.1, U2.12
- new net N$11: C_D2.1, U2.11, U2.14
- new net N$13: R_B4.2, U$14.P$3
- new net N$14: R1.1, R2.2, U1.4
- new net N$3: R4.1
- new net N$8: R_VM3.1, U2.6
- new net NFAULT: CR1.54, R_VM5.1, U2.8
- new net RESET: B1.3, CR1.7, C_NRST.1
- new net SW_VBST: C_NR3.1, L1.1, U1.2
- new net VBATT: C_3.3V7.1, C_3.3V9.1, C_NR2.1, U1.3
- net 3.3V: now also C_3.3V3.1, C_3.3V4.1, L2.1, R_B1.2, R_B2.2, R_PWR1.2, R_VM5.2, U$23.OUT, U2.1; no longer L1.1, R6.2
- net 5V: now also U$23.EN, U$23.IN; no longer C12.1, C15.1, C16.1, C6.1, C9.1, IC1.5, J3.4, J5.4, R2.1, R_VM4.1, U$12.L_VCC, U$12.R_VCC, U1.16, U2.11, U2.12, U2.14, U3.8
- net A3.3V: now also L2.2; no longer L1.2
- net AGND: now also U$22.2; no longer R_VM5.2, U1.8, U2.13, U3.5
- net CURRENT_SENSE: no longer C20.1, IC1.4, R_VM6.2
- net ENC_LA: no longer J5.6, U$12.L_CHA
- net ENC_LB: no longer J5.5, U$12.L_CHB
- net ENC_RA: no longer J3.6, U$12.R_CHA
- net ENC_RB: no longer J3.5, U$12.R_CHB
- net GND: now also B1.2, C_1.2, C_3.3V3.2, C_3.3V4.2, C_3.3V5.2, C_3.3V6.2, C_3.3V7.2, C_3.3V8.2, C_3.3V9.2, C_NR1.2, C_NR2.2, C_NRST.2, LED_PWR1.C, R2.1, R_B3.1, R_B4.1, U$16.1, U$22.1, U$23.GND, U1.1; no longer C12.2, C13.2, C15.2, C16.2, C3.2, C5.2, C6.2, C9.2, D1.1, IC1.2, J3.3, J5.3, R1.2, R8.1, R9.1, S1.1, S1.2, S3.1, U$12.L_GND, U$12.R_GND
- net I2C_SCL: no longer R4.1
- net INT: no longer CR1.28
- net N$1: now also C_NR1.1, U$23.NR/FB; no longer C13.1, U3.6
- net N$12: now also R_B3.2, U$15.P$3; no longer R2.2, U2.8
- net N$15: now also C_NR3.2, U1.6; no longer R9.2, U2.3
- net N$2: now also R_VM4.1, U2.3; no longer D1.3, R3.1, U1.5
- net N$4: now also R_B2.1, U$15.P$1; no longer CR1.10, S3.2
- net N$6: now also R_B1.1, U$14.P$1; no longer R6.1, S3.3
- net N$9: now also LED_PWR1.A, R_PWR1.1; no longer CR1.60, R1.1
- net REC_LD: no longer U1.3
- net REC_LF: no longer U1.4
- net REC_LH: no longer U1.14
- net REC_RD: no longer U1.2
- net REC_RF: no longer U1.1
- net REC_RH: no longer U1.15
- net V_BATT: no longer U3.2, U3.4
- net V_BATT_POWER: no longer U3.1, U3.3
Routing:
- removed copper zone on layer 15, net AGND
- removed copper zone on layer 1, net GND
- removed copper zone on layer 16, net GND
- removed copper zone on layer 2, net GND
Other:
- board size 93.9 x 75 mm -> 128.4 x 85.5 mm
