File: micromouse-main-board/micromouse-revB/micromouse_board_revB_V0.0.3.sch (EAGLE design)
At the start: 116 parts, among them IC1 LM321MFX, J3 HTSS-103-XX-XX-D, J5 HTSS-103-XX-XX-D, J6 HTSS-102-XX-XX-D, U1 SN74HC151DR, U2 DRV8848PWPR, U3 ACS712ELCTR-20A-T, U6 MPU-6000, X1 RASPI_GPIO_B+#_PIN

Commit message: power reg. added placement done
Parts:
- removed C12: 0.1 uF, micromouse-board-added-piconnector:CAP0603-CAP
- removed C13: 0.01uF, micromouse-board-added-piconnector:CAP0603-CAP
- removed C15: 10uF, micromouse-board-added-piconnector:CAP0603-CAP
- removed C16, C9: 2.2uF, micromouse-board-added-piconnector:CAP0603-CAP
- removed C20: 1000pF, micromouse-board-added-piconnector:CAP0603-CAP
- removed C3: 1.4 uF, micromouse-board-added-piconnector:CAP0603-CAP
- removed C5, C6: 0.1uF, micromouse-board-added-piconnector:CAP0603-CAP
- removed D1: (no value), diode:ZENER-DIODESOT23
- removed IC1: LM321MFX, micromouse-board-added-piconnector:LM321MFX
- removed J2: (no value), micromouse-board-added-piconnector:CONN_04
- removed J3, J5: HTSS-103-XX-XX-D, micromouse-board-added-piconnector:HTSS-103-XX-XX-D
- removed J6: HTSS-102-XX-XX-D, micromouse-board-added-piconnector:HTSS-102-XX-XX-D
- removed JP1, JP3: (no value), micromouse-board-added-piconnector:M02POLAR
- removed R3: 1k, rcl:R-US_R0805
- removed R6: 10k, rcl:R-US_M0805
- removed R8, R9: 500m, micromouse-board-added-piconnector:RESISTOR0805-RES
- removed R_VM6: 3.3k, micromouse-board-added-piconnector:RESISTOR0603-RES
- removed R_VM7: 1k, micromouse-board-added-piconnector:RESISTOR0603-RES
- removed S1: RESET, micromouse-board-added-piconnector:SWITCH-MOMENTARY-2SMD-4.6X2.8MM
- removed S3: (no value), micromouse-board-added-piconnector:SWITCH-SPSTPTH
- removed U3: ACS712ELCTR-20A-T, micromouse-board-added-piconnector:ACS712ELCTR-20A-T
- added B1: (no value), SparkFun-Retired:TAC_SWITCHSMD
- added C_1, C_3.3V4, C_D, C_NR1, C_NR2, C_NR3: 0.1uF, micromouse-board-added-piconnector:CAP0603-CAP
- added C_3.3V3, C_3.3V7, C_3.3V8, C_3.3V9, C_D1: 10uF, micromouse-board-added-piconnector:CAP0603-CAP
- added C_3.3V5, C_3.3V6, C_D2: 22uF, micromouse-board-added-piconnector:CAP0603-CAP
- added C_NRST: 0.1uF, SparkFun:CAP0603-CAP
- added L2: 10uH, micromouse-board-added-piconnector:INDUCTOR1007
- added LED_PWR1: green, micromouse-board-added-piconnector:LED1206
- added R_B1, R_B2: 47k, SparkFun-Passives:RESISTOR0603-RES
- added R_B3, R_B4: 1k, SparkFun-Passives:RESISTOR0603-RES
- added R_PWR1: 1k, micromouse-board-added-piconnector:RESISTOR0603-RES
- added R_VM3: 500m, micromouse-board-added-piconnector:RESISTOR0603-RES
- added U$10, U$5, U$6: 6P_HEADER, micro-motor:6P_HEADER
- added U$14, U$15: SPARKFUN-SPDT, micro-motor:SPARKFUN-SPDT
- added U$16, U$22: SPLITTER, splitter:SPLITTER
- added U$23: TPS73633(SOT-23), micromouse-board-added-piconnector:TPS73633(SOT-23)
- L1: value 10uH -> 4.7uH
- R1: value 1k -> 68k; device rcl:R-US_M0805 -> micromouse-board-added-piconnector:RESISTOR0603-RES
- R2: device micromouse-board-added-piconnector:RESISTOR0805-RES -> micromouse-board-added-piconnector:RESISTOR0603-RES
- R4, R5: value 10k -> 4.6k
- R_PWR: value 1k -> 500 Ohms
- R_VM2: value 25k -> 40k
- R_VM4: value 100k -> 500m
- R_VM5: value 100k -> 10k
- U$12: value MY_MM_MOTOR_MOUNT -> 6P_HEADER; device micromouse-board-added-piconnector:MY_MM_MOTOR_MOUNT -> micro-motor:6P_HEADER
- U1: value SN74HC151DR -> TPS561201DDCT; device micromouse-board-added-piconnector:SN74HC151DR -> micromouse-board-added-piconnector:TPS561201DDCT
Connections:
- net (USART1)_RX renamed USART1_RX
- net (USART1)_TX renamed USART1_TX
- removed net I_SENSE: U1.D6
- removed net LEFT_MOTOR_H: J5.2, JP1.1, U$12.L_MOTOR_A, U2.AOUT
- removed net LEFT_MOTOR_L: J5.1, JP1.2, U$12.L_MOTOR_B, U2.AOUT2
- removed net MUX_EN: CR1.PA11, U1.~G
- removed net N$20: R8.2, U2.BISEN
- removed net N$21: IC1.+IN, R_VM4.2, R_VM5.1
- removed net N$24: R_VM7.2, U3.VIOUT
- removed net N$31: C20.2, IC1.-IN, R_VM6.1, R_VM7.1
- removed net NRST: C5.1, CR1.NRST, S1.2
- removed net NSLEEP: U2.NSLEEP
- removed net PWM_MOTOR_1: CR1.PA1, J6.1, U2.AIN1
- removed net PWM_MOTOR_2: CR1.PA2, J6.2, U2.AIN2
- removed net PWM_MOTOR_3: CR1.PB0, J6.3, U2.BIN1
- removed net PWM_MOTOR_4: CR1.PB1, J6.4, U2.BIN2
- removed net RIGHT_MOTOR_H: J3.2, JP3.1, U$12.R_MOTOR_A, U2.BOUT1
- removed net RIGHT_MOTOR_L: J3.1, JP3.2, U$12.R_MOTOR_B, U2.BOUT2
- removed net SEL_A: U1.A
- removed net SEL_B: U1.B
- removed net SEL_C: U1.C
- removed net SENSOR_DEBUG: C3.1, J2.4, R3.2
- new net 6V: C_3.3V5.1, C_3.3V6.1, L1.2, R1.2, U$10.3, U$12.3, U$5.3, U$6.3, U1.EN
- new net BOOT0: CR1.BOOT0, U$14.P$2
- new net BOOT1: CR1.PB2, U$15.P$2
- new net BRIDGE_A_1: CR1.PA1, U2.AIN1
- new net BRIDGE_A_2: CR1.PA2, U2.AIN2
- new net BRIDGE_B_1: CR1.PB0, U2.BIN1
- new net BRIDGE_B_2: CR1.PB1, U2.BIN2
- new net M1_A: U$12.1, U$6.1, U2.AOUT
- new net M1_B: U$12.2, U$6.2, U2.AOUT2
- new net M1_ENC_A: U$12.4, U$6.4
- new net M1_ENC_B: U$12.5, U$6.5
- new net M2_A: U$10.1, U$5.1, U2.BOUT1
- new net M2_B: U$10.2, U$5.2, U2.BOUT2
- new net M2_ENC_A: U$10.5, U$5.4
- new net M2_ENC_B: U$10.4, U$5.5
- new net MGND: C_D.2, C_D1.2, C_D2.2, R_VM3.2, R_VM4.2, U$10.8, U$12.8, U$16.2, U$5.8, U$6.8, U2.GND
- new net N$10: C_D.1, C_D1.1, U2.VM
- new net N$11: C_D2.1, U2.VINT, U2.VREF
- new net N$13: R_B4.2, U$14.P$3
- new net N$14: R1.1, R2.2, U1.VFB
- new net N$3: R4.1
- new net N$8: R_VM3.1, U2.BISEN
- new net NFAULT: CR1.PD2, R_VM5.1, U2.NFAULT
- new net RESET: B1.3, CR1.NRST, C_NRST.1
- new net SW_VBST: C_NR3.1, L1.1, U1.SW
- new net VBATT: C_3.3V7.1, C_3.3V9.1, C_NR2.1, U1.VIN
- net 3.3V: now also C_3.3V3.1, C_3.3V4.1, L2.1, R_B1.2, R_B2.2, R_PWR1.2, R_VM5.2, U$23.OUT, U2.NSLEEP; no longer L1.1, R6.2
- net 5V: now also U$23.EN, U$23.IN; no longer C12.1, C15.1, C16.1, C6.1, C9.1, IC1.V+, J3.4, J5.4, R2.1, R_VM4.1, U$12.L_VCC, U$12.R_VCC, U1.VCC, U2.VINT, U2.VM, U2.VREF, U3.VCC
- net A3.3V: now also L2.2; no longer L1.2
- net AGND: now also U$22.2; no longer R_VM5.2, U1.GND, U2.GND, U3.GND
- net CURRENT_SENSE: no longer C20.1, IC1.OUT, R_VM6.2
- net ENC_LA: no longer J5.6, U$12.L_CHA
- net ENC_LB: no longer J5.5, U$12.L_CHB
- net ENC_RA: no longer J3.6, U$12.R_CHA
- net ENC_RB: no longer J3.5, U$12.R_CHB
- net GND: now also B1.2, C_1.2, C_3.3V3.2, C_3.3V4.2, C_3.3V5.2, C_3.3V6.2, C_3.3V7.2, C_3.3V8.2, C_3.3V9.2, C_NR1.2, C_NR2.2, C_NRST.2, LED_PWR1.C, R2.1, R_B3.1, R_B4.1, U$16.1, U$22.1, U$23.GND, U1.GND; no longer C12.2, C13.2, C15.2, C16.2, C3.2, C5.2, C6.2, C9.2, D1.A, IC1.V-, J3.3, J5.3, R1.2, R8.1, R9.1, S1.1, S3.O, U$12.L_GND, U$12.R_GND
- net I2C_SCL: no longer R4.1
- net INT: no longer CR1.PB2
- net N$1: now also C_NR1.1, U$23.NR/FB; no longer C13.1, U3.FILTER
- net N$12: now also R_B3.2, U$15.P$3; no longer R2.2, U2.NFAULT
- net N$15: now also C_NR3.2, U1.VBST; no longer R9.2, U2.AISEN
- net N$2: now also R_VM4.1, U2.AISEN; no longer D1.C, R3.1, U1.Y
- net N$4: now also R_B2.1, U$15.P$1; no longer CR1.PC2, S3.P
- net N$6: now also R_B1.1, U$14.P$1; no longer R6.1, S3.S
- net N$9: now also LED_PWR1.A, R_PWR1.1; no longer CR1.BOOT0, R1.1
- net REC_LD: no longer U1.D1
- net REC_LF: no longer U1.D0
- net REC_LH: no longer U1.D5
- net REC_RD: no longer U1.D2
- net REC_RF: no longer U1.D3
- net REC_RH: no longer U1.D4
- net V_BATT: no longer U3.IP+, U3.IP-_2
- net V_BATT_POWER: no longer U3.IP+_2, U3.IP-
Other:
- note added: "ADC12_IN8/TIM3_CH3 TIM8_CH3N"
- note added: "Boot & Reset Switches"
- note added: "C_D2 must be rated to atleast 6.3 V"
- note added: "DNI"
- note added: "I2C2_SCL/USART3_TX(9)"
- note added: "I2C2_SDA/USART3_RX(9)"
- note added: "IMU"
- note added: "JTCK- SWCLK"
- note added: "JTMS- SWDIO"
- note added: "PB2/BOOT1"
- note added: "SPI2_MISO/TIM1_CH2N USART3_RTS(9)/"
- note added: "SPI2_MOSI/I2S2_SD TIM1_CH3N(9)/"
- note added: "SPI2_NSS/I2S2_WS/ I2C2_SMBA/ USART3_CK"
- note added: "SPI2_SCK/I2S2_CK USART3_CTS(9)/ TIM1_CH1N"
- note added: "Test motors and encoders ----------------------"
- note added: "Two 3.7V Lipo"
- note added: "USART1_RX(9)/ TIM1_CH3(9)"
- note added: "USART1_TX(9)/ TIM1_CH2(9)"
- note added: "USART2_RTS(9) ADC123_IN1/ TIM5_CH2/TIM2_CH2(9)"
- note added: "USART2_TX(9)/TIM5_CH3 ADC123_IN2/ TIM2_CH3 (9)"
- note added: "VOUT = (0.768)*(1+ (R1/R2))"
- note removed: "ADC123_IN1/TIM2_CH2/TIM5_CH2"
- note removed: "ADC123_IN2/TIM5_CH3/TIM2_CH3"
- note removed: "Add beacon"
- note removed: "Analog Sensor Mux"
- note removed: "Batteries"
- note removed: "Reset Switch"
- note removed: "needs to be checked"
- moved on the sheet: C_GY_CP, C_GY_REG, C_GY_VDD, L1, R1, R2, R4, R5, R_VM4, R_VM5, TP1, TP2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
