File: micromouse-main-board/micromouse-revB/micromouse_board_revB_V0.0.5.sch (EAGLE design)
At the start: 110 parts, among them IC1 LM321MFX, J3 HTSS-103-XX-XX-D, J5 HTSS-103-XX-XX-D, J6 HTSS-102-XX-XX-D, U2 DRV8848PWPR, U3 ACS712ELCTR-20A-T, U6 MPU-6000, X1 RASPI_GPIO_B+#_PIN

Commit message: power reg. added placement done
Parts:
- removed C12: 0.1 uF, micromouse-board-added-piconnector:CAP0603-CAP
- removed C13: 0.01uF, micromouse-board-added-piconnector:CAP0603-CAP
- removed C15: 10uF, micromouse-board-added-piconnector:CAP0603-CAP
- removed C16: 2.2uF, micromouse-board-added-piconnector:CAP0603-CAP
- removed C20: 1000pF, micromouse-board-added-piconnector:CAP0603-CAP
- removed C5, C6, C_GY_REG, C_GY_VDD: 0.1uF, micromouse-board-added-piconnector:CAP0603-CAP
- removed C_GY_CP: 2.2nF, micromouse-board-added-piconnector:CAP0603-CAP
- removed IC1: LM321MFX, micromouse-board-added-piconnector:LM321MFX
- removed J5: HTSS-103-XX-XX-D, micromouse-board-added-piconnector:HTSS-103-XX-XX-D
- removed J6: HTSS-102-XX-XX-D, micromouse-board-added-piconnector:HTSS-102-XX-XX-D
- removed JP1, JP3: (no value), micromouse-board-added-piconnector:M02POLAR
- removed LED_PWR: green, micromouse-board-added-piconnector:LED1206
- removed R1: 1k, rcl:R-US_M0805
- removed R2: 10k, micromouse-board-added-piconnector:RESISTOR0805-RES
- removed R6: 10k, rcl:R-US_M0805
- removed R8, R9: 500m, micromouse-board-added-piconnector:RESISTOR0805-RES
- removed R_PWR, R_VM7: 1k, micromouse-board-added-piconnector:RESISTOR0603-RES
- removed R_VM6: 3.3k, micromouse-board-added-piconnector:RESISTOR0603-RES
- removed S1: RESET, micromouse-board-added-piconnector:SWITCH-MOMENTARY-2SMD-4.6X2.8MM
- removed S3: (no value), micromouse-board-added-piconnector:SWITCH-SPSTPTH
- removed U$1, U$2: JST_CONNECTOR_FEMALE, micromouse-board-added-piconnector:JST_CONNECTOR_FEMALE
- removed U$12: MY_MM_MOTOR_MOUNT, micromouse-board-added-piconnector:MY_MM_MOTOR_MOUNT
- removed U3: ACS712ELCTR-20A-T, micromouse-board-added-piconnector:ACS712ELCTR-20A-T
- added 3.3V_PWR, 5V_PWR1, 6V_PWR1: green, micromouse-board-added-piconnector:LED1206
- added B1: (no value), SparkFun-Retired:TAC_SWITCHSMD
- added C_3.3V5: 1uF, micromouse-board-added-piconnector:CAP0603-CAP
- added C_3.3V6, C_D1: 10uF, micromouse-board-added-piconnector:CAP0603-CAP
- added C_3.3V7, C_D, IMU_C1, IMU_C2: 0.1uF, micromouse-board-added-piconnector:CAP0603-CAP
- added C_D2: 2.2uF, micromouse-board-added-piconnector:CAP0603-CAP
- added C_NRST: 0.1uF, SparkFun:CAP0603-CAP
- added IMU_C3: 2.2nF, micromouse-board-added-piconnector:CAP0603-CAP
- added J2: JST_PH, B2B-PH-K-S_LF__SN_:B2B-PH-K-S(LF)(SN)
- added R_B1, R_B2: 47k, SparkFun-Passives:RESISTOR0603-RES
- added R_PWR1, R_PWR3, R_PWR4: 100 Ohm, micromouse-board-added-piconnector:RESISTOR0603-RES
- added R_VM3: 500m, micromouse-board-added-piconnector:RESISTOR0603-RES
- added TP10, TP11, TP7, TP8, TP9: (no value), micromouse-board-added-piconnector:TESTPOINTROUND2MM
- added U$14, U$15: SPARKFUN-SPDT, micro-motor:SPARKFUN-SPDT
- added U$16, U$22: SPLITTER, splitter:SPLITTER
- added U$23: BD60HC5WEFJ, BD33FC0WEFJ-E2:BD60HC5WEFJ
- added U$5, U$6: 6P_HEADER, micro-motor:6P_HEADER
- C1: value 1.1uF -> 0.01uF
- C4: value 0.01uF -> 0.1uF
- C8: value 4.7uF -> 1uF
- J3: value HTSS-103-XX-XX-D -> JST_PH; device micromouse-board-added-piconnector:HTSS-103-XX-XX-D -> B2B-PH-K-S_LF__SN_:B2B-PH-K-S(LF)(SN)
- L1: device micromouse-board-added-piconnector:INDUCTOR1007 -> SparkFun-Passives:INDUCTOR1007
- R4, R5: value 10k -> 4.6k
- R_ERF: value 10 -> 30 Ohms
- R_VM1: value 75k -> 70k
- R_VM2: value 25k -> 40k
- R_VM4: value 100k -> 500m
- R_VM5: value 100k -> 10k
Connections:
- net (USART1)_RX renamed USART1_RX
- net (USART1)_TX renamed USART1_TX
- removed net BATT_CONN: U$1.+, U$2.-
- removed net LEFT_MOTOR_H: J5.2, JP1.1, U$12.L_MOTOR_A, U2.AOUT
- removed net LEFT_MOTOR_L: J5.1, JP1.2, U$12.L_MOTOR_B, U2.AOUT2
- removed net MUX_EN: CR1.PA11
- removed net N$12: R2.2, U2.NFAULT
- removed net N$15: R9.2, U2.AISEN
- removed net N$20: R8.2, U2.BISEN
- removed net N$21: IC1.+IN, R_VM4.2, R_VM5.1
- removed net N$24: R_VM7.2, U3.VIOUT
- removed net N$27: LED_PWR.A, R_PWR.1
- removed net N$31: C20.2, IC1.-IN, R_VM6.1, R_VM7.1
- removed net NRST: C5.1, CR1.NRST, S1.2
- removed net NSLEEP: U2.NSLEEP
- removed net PWM_MOTOR_1: CR1.PA1, J6.1, U2.AIN1
- removed net PWM_MOTOR_2: CR1.PA2, J6.2, U2.AIN2
- removed net PWM_MOTOR_3: CR1.PB0, J6.3, U2.BIN1
- removed net PWM_MOTOR_4: CR1.PB1, J6.4, U2.BIN2
- removed net RIGHT_MOTOR_H: J3.2, JP3.1, U$12.R_MOTOR_A, U2.BOUT1
- removed net RIGHT_MOTOR_L: J3.1, JP3.2, U$12.R_MOTOR_B, U2.BOUT2
- removed net V_BATT_POWER: S2.S, U$2.+, U3.IP+_2, U3.IP-
- new net 6V: C_3.3V5.1, U$23.VO, U$5.3, U$6.3
- new net 6V_S: R_PWR3.2, U$23.VO_S
- new net BOOT0: CR1.BOOT0, U$14.P$2
- new net BOOT1: CR1.PB2, U$15.P$2
- new net BRIDGE_A_1: CR1.PA1, U2.AIN1
- new net BRIDGE_A_2: CR1.PA2, U2.AIN2
- new net BRIDGE_B_1: CR1.PB0, U2.BIN1
- new net BRIDGE_B_2: CR1.PB1, U2.BIN2
- new net M1_A: U$6.1, U2.AOUT
- new net M1_B: U$6.2, U2.AOUT2
- new net M1_ENC_A: TP7.P$1, U$6.4
- new net M1_ENC_B: TP8.P$1, U$6.5
- new net M2_A: U$5.1, U2.BOUT1
- new net M2_B: U$5.2, U2.BOUT2
- new net M2_ENC_A: TP9.P$1, U$5.4
- new net M2_ENC_B: TP10.P$1, U$5.5
- new net MGND: C_D.2, C_D1.2, C_D2.2, R_VM3.2, R_VM4.2, U$16.2, U$5.8, U$6.8, U2.GND
- new net N$10: C_D.1, C_D1.1, U2.VM
- new net N$11: C_D2.1, U2.VINT, U2.VREF
- new net N$14: 5V_PWR1.A, R_PWR1.1
- new net N$2: R_VM4.1, U2.AISEN
- new net N$3: J2.1, J3.2
- new net N$8: R_VM3.1, U2.BISEN
- new net NFAULT: CR1.PD2, R_VM5.1, U2.NFAULT
- new net RESET: B1.3, CR1.NRST, C_NRST.1
- new net VBAT_POWER: J3.1, S2.S
- net 3.3V: now also IMU_C2.1, R_B1.2, R_B2.2, R_PWR4.2, R_VM5.2, U2.NSLEEP; no longer C_GY_VDD.1, R6.2
- net 5V: now also R_PWR1.2; no longer C12.1, C15.1, C16.1, C6.1, IC1.V+, J3.4, J5.4, R2.1, R_PWR.2, R_VM4.1, U$12.L_VCC, U$12.R_VCC, U2.VINT, U2.VM, U2.VREF, U3.VCC
- net AGND: now also IMU_C1.2, IMU_C2.2, IMU_C3.2, U$22.2; no longer C_GY_CP.2, C_GY_REG.2, C_GY_VDD.2, R_VM5.2, U2.GND, U3.GND
- net CURRENT_SENSE: no longer C20.1, IC1.OUT, R_VM6.2
- net ENC_LA: no longer J5.6, U$12.L_CHA
- net ENC_LB: no longer J5.5, U$12.L_CHB
- net ENC_RA: no longer J3.6, U$12.R_CHA
- net ENC_RB: no longer J3.5, U$12.R_CHB
- net GND: now also 3.3V_PWR.C, 5V_PWR1.C, 6V_PWR1.C, B1.2, C_3.3V5.2, C_3.3V6.2, C_3.3V7.2, C_NRST.2, J2.2, TP11.P$1, U$14.P$3, U$15.P$3, U$16.1, U$22.1, U$23.EPAD, U$23.GND, U$23.N.C_1, U$23.N.C_2, U$23.N.C_3; no longer C12.2, C13.2, C15.2, C16.2, C5.2, C6.2, IC1.V-, J3.3, J5.3, LED_PWR.C, R1.2, R8.1, R9.1, S1.1, S3.O, U$1.-, U$12.L_GND, U$12.R_GND
- net INT: no longer CR1.PB2
- net N$1: now also 3.3V_PWR.A, R_PWR4.1; no longer C13.1, U3.FILTER
- net N$28: now also IMU_C1.1; no longer C_GY_REG.1
- net N$29: now also IMU_C3.1; no longer C_GY_CP.1
- net N$4: now also R_B2.1, U$15.P$1; no longer CR1.PC2, S3.P
- net N$6: now also R_B1.1, U$14.P$1; no longer R6.1, S3.S
- net N$9: now also 6V_PWR1.A, R_PWR3.1; no longer CR1.BOOT0, R1.1
- net V_BATT: now also C_3.3V6.1, C_3.3V7.1, U$23.EN, U$23.VCC; no longer U3.IP+, U3.IP-_2
Other:
- note added: "+/-1% output voltage accuracy"
- note added: "ADC12_IN8/TIM3_CH3 TIM8_CH3N"
- note added: "Boot & Reset Switches"
- note added: "C3 needs to be rated for 50 V"
- note added: "C_D2 must be rated to atleast 6.3 V"
- note added: "I2C2_SCL/USART3_TX(9)"
- note added: "I2C2_SDA/USART3_RX(9)"
- note added: "IMU"
- note added: "JTCK- SWCLK"
- note added: "JTMS- SWDIO"
- note added: "Make 1/2 W resistors"
- note added: "PB2/BOOT1"
- note added: "PROGRAMMING DEBUG HEADER"
- note added: "SPI2_MISO/TIM1_CH2N USART3_RTS(9)/"
- note added: "SPI2_MOSI/I2S2_SD TIM1_CH3N(9)/"
- note added: "SPI2_NSS/I2S2_WS/ I2C2_SMBA/ USART3_CK"
- note added: "SPI2_SCK/I2S2_CK USART3_CTS(9)/ TIM1_CH1N"
- note added: "Switch to JST PH Connectors"
- note added: "Test motors and encoders"
- note added: "Two 3.7V Lipo"
- note added: "USART1_RX(9)/ TIM1_CH3(9)"
- note added: "USART1_TX(9)/ TIM1_CH2(9)"
- note added: "USART2_RTS(9) ADC123_IN1/ TIM5_CH2/TIM2_CH2(9)"
- note added: "USART2_TX(9)/TIM5_CH3 ADC123_IN2/ TIM2_CH3 (9)"
- note added: "V_mcu = V_bat * (40/(40 + 70))"
- note removed: "ADC123_IN1/TIM2_CH2/TIM5_CH2"
- note removed: "ADC123_IN2/TIM5_CH3/TIM2_CH3"
- note removed: "Add beacon"
- note removed: "Analog Sensor Mux"
- note removed: "Batteries"
- note removed: "Note: Enable Pins need to be changed"
- note removed: "PROGRAMMING/DEBUG HEADER"
- note removed: "R_PWR needs to be a HIGH POWER resistor"
- note removed: "Reset Switch"
- note removed: "V_mcu = V_bat * (1/4)"
- moved on the sheet: L1, R4, R5, R_VM4, R_VM5, TP1, TP2, TP3, TP4, TP5, TP6, U6
