File: micromouse-main-board/micromouse-revB/micromouse_board_revB_V0.0.10.brd (EAGLE design)
At the start: 128.4 x 85.5 mm, 117 parts, among them J2 JST_PH, J3 JST_PH, U2 DRV8848PWPR, U6 MPU-6000, X1 RASPI_GPIO_B+#_PIN

Commit message: planes seem to be layed nicely
Parts:
- removed 5V_PWR1, 6V_PWR1: green, micromouse-board-added-piconnector:LED-1206
- removed TP1, TP2, TP3, TP4, TP5, TP6: (no value), micromouse-board-added-piconnector:TESTPOINT_ROUND_2MM
- added 5V_PWR, 6V_PWR: green, micromouse-board-added-piconnector:LED-1206
- added T1, T2, T3, T4, T5, T6, TP12, TP13: (no value), micromouse-board-added-piconnector:TESTPOINT_ROUND_2MM
- C1: value 0.01uF -> 10nF
- R_ERF: value 30 Ohms -> 30
- moved C_NRST1 293.4 mm to (42.2, 22.6), turned to 270 degrees
- moved C_NRST2 286.9 mm to (42.1, 16.9), turned to 270 degrees
- moved B2 281.4 mm to (37.5, 21.8), turned to 180 degrees
- moved B3 281.0 mm to (37.5, 16.1), turned to 180 degrees
- moved R_RLH 43.2 mm to (87.8, 50.2)
- moved R_VM2 26.5 mm to (55.3, 19.2), turned to 180 degrees
- moved R5 26.3 mm to (47.2, 19.6), turned to 90 degrees
- moved R_VM1 26.3 mm to (54.4, 22.0), turned to 90 degrees
- moved C_5V1 26.1 mm to (-4.48, 38.9), turned to 270 degrees
- moved R4 22.1 mm to (49.2, 19.6), turned to 90 degrees
- moved C_BAT2 14.0 mm to (-13.4, 39.4)
- moved R_B1 12.0 mm to (51.1, 0.67), turned to 270 degrees
- moved U$15 11.8 mm to (55.1, 0.26), turned to 270 degrees
- moved NMOS3 11.6 mm to (60.3, 8.92)
- moved R_B2 11.5 mm to (59.3, 0.69), turned to 270 degrees
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Connections:
- removed net CURRENT_SENSE: CR1.20
- removed net ENC_LA: CR1.40
- removed net ENC_LB: CR1.39
- removed net ENC_RA: CR1.37
- removed net ENC_RB: CR1.38
- removed net N$10: C_D.1, C_D1.1, U2.12
- net 3.3V: no longer C1.2, C8.2, CR1.13, IMU_C2.1, U6.13
- net 6V: now also C_D.1, C_D1.1, U2.12
- net A3.3V: now also C1.2, C8.2, CR1.13, IMU_C2.1, U6.13
- net AGND: now also C1.1, C8.1, CR1.12, TP12.P$1
- net GND: now also 5V_PWR.C, 6V_PWR.C, B1.1, TP13.P$1; no longer 5V_PWR1.C, 6V_PWR1.C, C1.1, C8.1, CR1.12, TP11.P$1
- net INT: now also CR1.56
- net M1_ENC_A: now also CR1.37
- net M1_ENC_B: now also CR1.38
- net M2_ENC_A: now also CR1.40
- net M2_ENC_B: now also CR1.39
- net MGND: now also TP11.P$1
- net N$14: now also 5V_PWR.A; no longer 5V_PWR1.A
- net N$9: now also 6V_PWR.A; no longer 6V_PWR1.A
- net REC_LD: now also T3.P$1; no longer TP2.P$1
- net REC_LF: now also T1.P$1; no longer TP1.P$1
- net REC_LH: now also T2.P$1; no longer TP4.P$1
- net REC_RD: now also T4.P$1; no longer TP5.P$1
- net REC_RF: now also T6.P$1; no longer TP6.P$1
- net REC_RH: now also T5.P$1; no longer TP3.P$1
- net RESET: now also B1.4
Routing:
- net A3.3V: track 0.00 -> 231.2 mm, vias 0 -> 15
- net AGND: track 0.00 -> 156.1 mm, vias 0 -> 4
- net 6V: track 0.00 -> 125.0 mm
- net 3.3V: track 0.00 -> 110.8 mm, vias 0 -> 2
- net GND: track 0.00 -> 55.8 mm, vias 0 -> 34
- net M1_A: track 0.00 -> 40.8 mm
- net D_EM: track 0.00 -> 40.0 mm
- net M1_ENC_A: track 0.00 -> 37.5 mm, vias 0 -> 1
- net RESET: track 0.00 -> 33.1 mm, vias 0 -> 2
- net M1_ENC_B: track 0.00 -> 33.0 mm, vias 0 -> 1
- net BOOT1: track 0.00 -> 32.4 mm, vias 0 -> 2
- net M1_B: track 0.00 -> 30.5 mm, vias 0 -> 1
- net M2_ENC_B: track 0.00 -> 29.0 mm, vias 0 -> 1
- net M2_B: track 0.00 -> 28.9 mm, vias 0 -> 1
- net BRIDGE_B_1: track 0.00 -> 28.4 mm, vias 0 -> 1
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- added copper zone on layer 1, net 3.3V
- added copper zone on layer 1, net 5V
- added copper zone on layer 1, net 6V
- added copper zone on layer 16, net A3.3V
- added copper zone on layer 16, net AGND
- added copper zone on layer 1, net GND
- added copper zone on layer 16, net GND
- added copper zone on layer 1, net MGND
- added copper zone on layer 1, net V_BATT
Other:
- board text added: "1"
- board text added: "2"
- board text added: "3"
- board text added: "4"
- board text added: "5"
- board text added: "6"
- board text added: "A. Spain"
- board text added: "AGND"
- board text added: "BAT 1"
- board text added: "BAT 2"
- board text added: "Bottom Planes ------------ 1. AGND 2. GND 3. A3.3V"
- board text added: "IMU"
- board text added: "L"
- board text added: "M1 ENC A"
- board text added: "M1 ENC B"
- board text added: "M2 ENC A"
- board text added: "M2 ENC B"
- board text added: "MGND"
- board text added: "MOTOR 1"
- board text added: "MOTOR CTRL"
- board text added: "MOTOR2"
- board text added: "OFF"
- board text added: "ON"
- board text added: "PRGM 1"
- board text added: "PRGM 2"
- board text added: "PWR SWITCh"
- board text added: "Serial Wire"
- board text added: "Top Planes --------- 1. 5V, GND 2.MGND 3.3.3V 4. 6V 5. 6. V_BATT"
- board text added: "UGA 2020 Robotics Club"
- board text added: "USART"
- board text added: "X"
- board text added: "Y"
- board text added: "Z"
