File: micromouse-main-board/micromouse-revB/micromouse_board_revB_V0.0.10.sch (EAGLE design)
At the start: 117 parts, among them J2 JST_PH, J3 JST_PH, U2 DRV8848PWPR, U6 MPU-6000, X1 RASPI_GPIO_B+#_PIN

Commit message: planes seem to be layed nicely
Parts:
- removed TP1, TP2, TP3, TP4, TP5, TP6: (no value), micromouse-board-added-piconnector:TESTPOINTROUND2MM
- added T1, T2, T3, T4, T5, T6, TP12, TP13: (no value), micromouse-board-added-piconnector:TESTPOINTROUND2MM
- C1: value 0.01uF -> 10nF
- R_ERF: value 30 Ohms -> 30
- renumbered 5V_PWR1 to 5V_PWR, 6V_PWR1 to 6V_PWR
Connections:
- removed net CURRENT_SENSE: CR1.PA4
- removed net ENC_LA: CR1.PC9
- removed net ENC_LB: CR1.PC8
- removed net ENC_RA: CR1.PC6
- removed net ENC_RB: CR1.PC7
- removed net N$10: C_D.1, C_D1.1, U2.VM
- net 3.3V: no longer C1.2, C8.2, CR1.VDDA, IMU_C2.1, U6.VDD
- net 6V: now also C_D.1, C_D1.1, U2.VM
- net A3.3V: now also C1.2, C8.2, CR1.VDDA, IMU_C2.1, U6.VDD
- net AGND: now also C1.1, C8.1, CR1.VSSA, TP12.P$1
- net GND: now also B1.1, TP13.P$1; no longer C1.1, C8.1, CR1.VSSA, TP11.P$1
- net INT: now also CR1.PB4
- net M1_ENC_A: now also CR1.PC6
- net M1_ENC_B: now also CR1.PC7
- net M2_ENC_A: now also CR1.PC9
- net M2_ENC_B: now also CR1.PC8
- net MGND: now also TP11.P$1
- net REC_LD: now also T3.P$1; no longer TP2.P$1
- net REC_LF: now also T1.P$1; no longer TP1.P$1
- net REC_LH: now also T2.P$1; no longer TP4.P$1
- net REC_RD: now also T4.P$1; no longer TP5.P$1
- net REC_RF: now also T6.P$1; no longer TP6.P$1
- net REC_RH: now also T5.P$1; no longer TP3.P$1
- net RESET: now also B1.4
Other:
- note added: "Make sure these Caps are rated for atleast 10 V"
- note added: "SPI3_MISO remap to PB4 / TIM3_CH1 SPI1_MISO"
- note added: "Test points for motors and encoders"
- note added: "V_bat = ((40+70)/(40)) * V_mcu V_mcu should not exceed 2.90V"
- note removed: "Changelog -------------------------------------- 06/08/2019 - Added MCU, board outline and IR sensors and receivers. 07/17/2019 - Added Motor Driver, MUX for sensor input, Current Sensor, picked GPIO to use for MUX select, picked ADC in to route MUX to. 07/18/2019 - Programming/debug header added. 07/27/2019 - Connected sensors and added mpu600 and power monitor"
- note removed: "Notes -------------------------------------- Add product specs and notes on 'Guide' layer Use GND symbol and VCC symbol for ground and power respectively. (Rather than tags)"
- note removed: "SWITCH TO SET MODE"
- note removed: "Test motors and encoders"
- note removed: "V_mcu = V_bat * (40/(40 + 70))"
