File: micromouse-main-board/micromouse-revB/micromouse_board_revB_V0.0.4.brd (EAGLE design)
At the start: 41 x 75 mm, 110 parts, among them IC1 LM321MFX, J3 HTSS-103-XX-XX-D, J5 HTSS-103-XX-XX-D, J6 HTSS-102-XX-XX-D, U2 DRV8848PWPR, U3 ACS712ELCTR-20A-T, U6 MPU-6000, X1 RASPI_GPIO_B+#_PIN

Commit message: power reg. added placement done
Parts:
- removed C12: 0.1 uF, micromouse-board-added-piconnector:0603-CAP
- removed C13: 0.01uF, micromouse-board-added-piconnector:0603-CAP
- removed C15: 10uF, micromouse-board-added-piconnector:0603-CAP
- removed C16: 2.2uF, micromouse-board-added-piconnector:0603-CAP
- removed C20: 1000pF, micromouse-board-added-piconnector:0603-CAP
- removed C5, C6, C_GY_REG, C_GY_VDD: 0.1uF, micromouse-board-added-piconnector:0603-CAP
- removed C_GY_CP: 2.2nF, micromouse-board-added-piconnector:0603-CAP
- removed IC1: LM321MFX, micromouse-board-added-piconnector:SOT23-5
- removed J5: HTSS-103-XX-XX-D, micromouse-board-added-piconnector:HTSS-103-XX-XX-D
- removed J6: HTSS-102-XX-XX-D, micromouse-board-added-piconnector:HTSS-102-XX-XX-D
- removed JP1, JP3: (no value), micromouse-board-added-piconnector:MOLEX-1X2
- removed LED_PWR: green, micromouse-board-added-piconnector:LED-1206
- removed R1: 1k, rcl:M0805
- removed R2: 10k, micromouse-board-added-piconnector:0805
- removed R6: 10k, rcl:M0805
- removed R8, R9: 500m, micromouse-board-added-piconnector:0805
- removed R_PWR, R_VM7: 1k, micromouse-board-added-piconnector:0603-RES
- removed R_VM6: 3.3k, micromouse-board-added-piconnector:0603-RES
- removed S1: RESET, micromouse-board-added-piconnector:TACTILE_SWITCH_SMD_4.6X2.8MM
- removed S3: (no value), micromouse-board-added-piconnector:SWITCH-SPDT
- removed U$1, U$2: JST_CONNECTOR_FEMALE, micromouse-board-added-piconnector:JST_CONNECTOR_FEMALE
- removed U$12: MY_MM_MOTOR_MOUNT, micromouse-board-added-piconnector:MY_MM_MOTOR_MOUNT
- removed U3: ACS712ELCTR-20A-T, micromouse-board-added-piconnector:SOIC127P600X175-8N
- added 3.3V_PWR, 5V_PWR1, 6V_PWR1: green, micromouse-board-added-piconnector:LED-1206
- added B1: (no value), SparkFun-Retired:TACTILE-SWITCH-SMD
- added C_3.3V5: 1uF, micromouse-board-added-piconnector:0603-CAP
- added C_3.3V6, C_D1: 10uF, micromouse-board-added-piconnector:0603-CAP
- added C_3.3V7, C_D, IMU_C1, IMU_C2: 0.1uF, micromouse-board-added-piconnector:0603-CAP
- added C_D2: 2.2uF, micromouse-board-added-piconnector:0603-CAP
- added C_NRST: 0.1uF, SparkFun:0603-CAP
- added IMU_C3: 2.2nF, micromouse-board-added-piconnector:0603-CAP
- added J2: B2B-PH-K-S(LF)(SN), B2B-PH-K-S_LF__SN_:JST_B2B-PH-K-S(LF)(SN)
- added R_B1, R_B2: 47k, SparkFun-Passives:0603-RES
- added R_PWR1, R_PWR3, R_PWR4: 100 Ohm, micromouse-board-added-piconnector:0603-RES
- added R_VM3: 500m, micromouse-board-added-piconnector:0603-RES
- added TP10, TP11, TP7, TP8, TP9: (no value), micromouse-board-added-piconnector:TESTPOINT_ROUND_2MM
- added U$14, U$15: SPARKFUN-SPDT, micro-motor:SPDT
- added U$16, U$22: SPLITTER, splitter:SPLITTER
- added U$23: BD60HC5WEFJ, BD33FC0WEFJ-E2:SOIC127P600X100-9N
- added U$5, U$6: 6P_HEADER, micro-motor:6P_HEADER
- C1: value 1.1uF -> 0.01uF
- C4: value 0.01uF -> 0.1uF
- C8: value 4.7uF -> 1uF
- J3: value HTSS-103-XX-XX-D -> B2B-PH-K-S(LF)(SN); device micromouse-board-added-piconnector:HTSS-103-XX-XX-D -> B2B-PH-K-S_LF__SN_:JST_B2B-PH-K-S(LF)(SN)
- L1: device micromouse-board-added-piconnector:1007 -> SparkFun-Passives:1007
- R4, R5: value 10k -> 4.6k
- R_ERF: value 10 -> 30 Ohms
- R_VM1: value 75k -> 70k
- R_VM2: value 25k -> 40k
- R_VM4: value 100k -> 500m
- R_VM5: value 100k -> 10k
- moved R4 71.2 mm to (69.6, 28.2), turned to 270 degrees
- moved R5 70.5 mm to (72.1, 28.2), turned to 270 degrees
- moved U6 69.5 mm to (73.4, 34.4), turned to 90 degrees
- moved TP1 43.8 mm to (55.0, 72.1)
- moved R_VM1 43.5 mm to (45.5, 46.7)
- moved R_VM2 43.3 mm to (45.5, 43.8)
- moved R_RLF 42.0 mm to (59.3, 74.0)
- moved L1 35.5 mm to (-10.4, 14.3)
- moved J3 34.3 mm to (-4.45, 56.6), turned to 90 degrees
- moved C21 33.8 mm to (63.1, 20.0), turned to 0 degrees
- moved C_3.3V2 32.3 mm to (-1.25, 9.90), turned to 0 degrees
- moved R_RLH 30.1 mm to (47.6, 34.5)
- moved R_RRD 29.1 mm to (92.0, 26.2), turned to 0 degrees
- moved C18 29.1 mm to (57.0, 19.9), flipped to the top
- moved R_ED_PD 27.6 mm to (90.9, 42.9), turned to 180 degrees
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Connections:
- net (USART1)_RX renamed USART1_RX
- net (USART1)_TX renamed USART1_TX
- removed net BATT_CONN: U$1.+, U$2.-
- removed net LEFT_MOTOR_H: J5.2, JP1.1, U$12.L_MOTOR_A, U2.2
- removed net LEFT_MOTOR_L: J5.1, JP1.2, U$12.L_MOTOR_B, U2.4
- removed net MUX_EN: CR1.44
- removed net N$12: R2.2, U2.8
- removed net N$15: R9.2, U2.3
- removed net N$20: R8.2, U2.6
- removed net N$21: IC1.1, R_VM4.2, R_VM5.1
- removed net N$24: R_VM7.2, U3.7
- removed net N$27: LED_PWR.A, R_PWR.1
- removed net N$31: C20.2, IC1.3, R_VM6.1, R_VM7.1
- removed net NRST: C5.1, CR1.7, S1.3, S1.4
- removed net NSLEEP: U2.1
- removed net PWM_MOTOR_1: CR1.15, J6.1, U2.16
- removed net PWM_MOTOR_2: CR1.16, J6.2, U2.15
- removed net PWM_MOTOR_3: CR1.26, J6.3, U2.9
- removed net PWM_MOTOR_4: CR1.27, J6.4, U2.10
- removed net RIGHT_MOTOR_H: J3.2, JP3.1, U$12.R_MOTOR_A, U2.7
- removed net RIGHT_MOTOR_L: J3.1, JP3.2, U$12.R_MOTOR_B, U2.5
- removed net V_BATT_POWER: S2.3, U$2.+, U3.1, U3.3
- new net 6V: C_3.3V5.1, U$23.1, U$5.3, U$6.3
- new net 6V_S: R_PWR3.2, U$23.2
- new net BOOT0: CR1.60, U$14.P$2
- new net BOOT1: CR1.28, U$15.P$2
- new net BRIDGE_A_1: CR1.15, U2.16
- new net BRIDGE_A_2: CR1.16, U2.15
- new net BRIDGE_B_1: CR1.26, U2.9
- new net BRIDGE_B_2: CR1.27, U2.10
- new net M1_A: U$6.1, U2.2
- new net M1_B: U$6.2, U2.4
- new net M1_ENC_A: TP7.P$1, U$6.4
- new net M1_ENC_B: TP8.P$1, U$6.5
- new net M2_A: U$5.1, U2.7
- new net M2_B: U$5.2, U2.5
- new net M2_ENC_A: TP9.P$1, U$5.4
- new net M2_ENC_B: TP10.P$1, U$5.5
- new net MGND: C_D.2, C_D1.2, C_D2.2, R_VM3.2, R_VM4.2, U$16.2, U$5.6, U$6.6, U2.13
- new net N$10: C_D.1, C_D1.1, U2.12
- new net N$11: C_D2.1, U2.11, U2.14
- new net N$14: 5V_PWR1.A, R_PWR1.1
- new net N$2: R_VM4.1, U2.3
- new net N$8: R_VM3.1, U2.6
- new net NFAULT: CR1.54, R_VM5.1, U2.8
- new net RESET: B1.3, CR1.7, C_NRST.1
- new net V_BATT_RAW: S2.3
- net 3.3V: now also IMU_C2.1, R_B1.2, R_B2.2, R_PWR4.2, R_VM5.2, U2.1; no longer C_GY_VDD.1, R6.2
- net 5V: now also R_PWR1.2; no longer C12.1, C15.1, C16.1, C6.1, IC1.5, J3.4, J5.4, R2.1, R_PWR.2, R_VM4.1, U$12.L_VCC, U$12.R_VCC, U2.11, U2.12, U2.14, U3.8
- net AGND: now also IMU_C1.2, IMU_C2.2, IMU_C3.2, U$22.2; no longer C_GY_CP.2, C_GY_REG.2, C_GY_VDD.2, R_VM5.2, U2.13, U3.5
- net CURRENT_SENSE: no longer C20.1, IC1.4, R_VM6.2
- net ENC_LA: no longer J5.6, U$12.L_CHA
- net ENC_LB: no longer J5.5, U$12.L_CHB
- net ENC_RA: no longer J3.6, U$12.R_CHA
- net ENC_RB: no longer J3.5, U$12.R_CHB
- net GND: now also 3.3V_PWR.C, 5V_PWR1.C, 6V_PWR1.C, B1.2, C_3.3V5.2, C_3.3V6.2, C_3.3V7.2, C_NRST.2, TP11.P$1, U$14.P$3, U$15.P$3, U$16.1, U$22.1, U$23.3, U$23.4, U$23.6, U$23.7, U$23.9; no longer C12.2, C13.2, C15.2, C16.2, C5.2, C6.2, IC1.2, J3.3, J5.3, LED_PWR.C, R1.2, R8.1, R9.1, S1.1, S1.2, S3.1, U$1.-, U$12.L_GND, U$12.R_GND
- net INT: no longer CR1.28
- net N$1: now also 3.3V_PWR.A, R_PWR4.1; no longer C13.1, U3.6
- net N$28: now also IMU_C1.1; no longer C_GY_REG.1
- net N$29: now also IMU_C3.1; no longer C_GY_CP.1
- net N$4: now also R_B2.1, U$15.P$1; no longer CR1.10, S3.2
- net N$6: now also R_B1.1, U$14.P$1; no longer R6.1, S3.3
- net N$9: now also 6V_PWR1.A, R_PWR3.1; no longer CR1.60, R1.1
- net V_BATT: now also C_3.3V6.1, C_3.3V7.1, U$23.5, U$23.8; no longer U3.2, U3.4
Other:
- board size 41 x 75 mm -> 128.4 x 85.5 mm
- board text added: "3.3V"
- board text added: "BOOT0"
- board text added: "BOOT1"
- board text added: "GND"
- board text removed: "BULLBOTS UGA 2019"

Commit message: planes seem to be layed nicely
Parts:
- added B2, B3: (no value), SparkFun-Retired:TACTILE-SWITCH-SMD
- added C_NRST1, C_NRST2: 0.1uF, SparkFun:0603-CAP
Connections:
- new net PRGM_1: B2.3, B2.4, CR1.10, C_NRST1.1
- new net PRGM_2: B3.3, B3.4, CR1.11, C_NRST2.1
- net GND: now also B2.1, B2.2, B3.1, B3.2, C_NRST1.2, C_NRST2.2
Other:
- board text added: "RESET"
Changed lines of the file:
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@@
 <text x="46.228" y="2.54" size="1.27" layer="21">GND</text>
 <text x="46.228" y="-4.826" size="1.27" layer="21">3.3V</text>
+<text x="38.25" y="58.15" size="1.778" layer="25" font="vector">RESET</text>
 </plain>
 <attributes>
@@
 <class number="5" name="3.3V" width="0.508" drill="0.254">
 <clearance class="5" value="0.254"/>
+</class>
+<class number="6" name="GND" width="0.508" drill="0.254">
+<clearance class="6" value="0.254"/>
 </class>
 </classes>
@@
 <attribute name="PACKAGE" value="None" x="-4.45" y="56.6" size="1.016" layer="27" rot="R90" display="off"/>
 </element>
+<element name="B2" library="SparkFun-Retired" package="TACTILE-SWITCH-SMD" value="" x="-88.75" y="-229.65" smashed="yes">
+<attribute name="NAME" x="-89.639" y="-227.872" size="0.4064" layer="25"/>
+<attribute name="PROD_ID" value="SWCH-08247" x="-88.75" y="-229.65" size="1.778" layer="27" display="off"/>
+<attribute name="VALUE" x="-89.639" y="-231.682" size="0.4064" layer="27"/>
+</element>
+<element name="C_NRST1" library="SparkFun" package="0603-CAP" value="0.1uF" x="-90.8" y="-233.65" smashed="yes">
+<attribute name="NAME" x="-91.689" y="-232.888" size="0.4064" layer="25" font="vector"/>
+<attribute name="VALUE" x="-91.816" y="-234.793" size="0.4064" layer="27" font="vector"/>
+</element>
+<element name="B3" library="SparkFun-Retired" package="TACTILE-SWITCH-SMD" value="" x="-88.75" y="-237.95" smashed="yes">
+<attribute name="NAME" x="-89.639" y="-236.172" size="0.4064" layer="25"/>
+<attribute name="PROD_ID" value="SWCH-08247" x="-88.75" y="-237.95" size="1.778" layer="27" display="off"/>
+<attribute name="VALUE" x="-89.639" y="-239.982" size="0.4064" layer="27"/>
+</element>
+<element name="C_NRST2" library="SparkFun" package="0603-CAP" value="0.1uF" x="-90.8" y="-241.95" smashed="yes">
+<attribute name="NAME" x="-91.689" y="-241.188" size="0.4064" layer="25" font="vector"/>
+<attribute name="VALUE" x="-91.816" y="-243.093" size="0.4064" layer="27" font="vector"/>
+</element>
 </elements>
 <signals>
@@
 <contactref element="CR1" pad="31"/>
 <contactref element="C23" pad="1"/>
+<contactref element="B2" pad="2"/>
+<contactref element="B2" pad="1"/>
+<contactref element="C_NRST1" pad="2"/>
+<contactref element="B3" pad="1"/>
+<contactref element="B3" pad="2"/>
+<contactref element="C_NRST2" pad="2"/>
 <wire x1="92.025" y1="37.001" x2="91.781" y2="42.937" width="0" layer="19" extent="1-1"/>
 <wire x1="94.205" y1="35.99" x2="92.025" y2="37.001" width="0" layer="19" extent="1-1"/>
@@
 <wire x1="-8.14" y1="61.87" x2="-16.73" y2="58.43" width="0" layer="19" extent="1-1"/>
 <wire x1="-5.87" y1="61.97" x2="-8.14" y2="61.87" width="0" layer="19" extent="1-1"/>
+<wire x1="-85.956" y1="-227.745" x2="-19.27" y2="15.25" width="0" layer="19" extent="1-1"/>
+<wire x1="-91.544" y1="-227.745" x2="-85.956" y2="-227.745" width="0" layer="19" extent="1-1"/>
+<wire x1="-89.95" y1="-233.65" x2="-91.544" y2="-227.745" width="0" layer="19" extent="1-1"/>
+<wire x1="-91.544" y1="-236.045" x2="-89.95" y2="-233.65" width="0" layer="19" extent="1-1"/>
+<wire x1="-85.956" y1="-236.045" x2="-89.95" y2="-233.65" width="0" layer="19" extent="1-1"/>
+<wire x1="-89.95" y1="-241.95" x2="-91.544" y2="-236.045" width="0" layer="19" extent="1-1"/>
 </signal>
 <signal name="5V">
@@
 <contactref element="B1" pad="3"/>
 <contactref element="CR1" pad="7"/>
-<wire x1="36.835" y1="53.868" x2="36.7" y2="48.8" width="0" layer="19" extent="1-1"/>
-<wire x1="54.1719" y1="35.207" x2="36.835" y2="53.868" width="0" layer="19" extent="1-1"/>
+<wire x1="36.7" y1="48.8" x2="36.835" y2="53.868" width="0" layer="19" extent="1-1"/>
+<wire x1="54.1719" y1="35.207" x2="36.7" y2="48.8" width="0" layer="19" extent="1-1"/>
 </signal>
 <signal name="BOOT1">
@@
 <wire x1="-13.438" y1="36.576" x2="-13.55" y2="22.098" width="0" layer="19" extent="1-1"/>
 </signal>
+<signal name="PRGM_2">
+<contactref element="CR1" pad="11"/>
+<contactref element="B3" pad="4"/>
+<contactref element="B3" pad="3"/>
+<contactref element="C_NRST2" pad="1"/>
+<wire x1="-85.956" y1="-239.855" x2="54.1719" y2="33.207" width="0" layer="19" extent="1-1"/>
+<wire x1="-91.544" y1="-239.855" x2="-85.956" y2="-239.855" width="0" layer="19" extent="1-1"/>
+<wire x1="-91.65" y1="-241.95" x2="-91.544" y2="-239.855" width="0" layer="19" extent="1-1"/>
+</signal>
+<signal name="PRGM_1">
+<contactref element="CR1" pad="10"/>
+<contactref element="B2" pad="3"/>
+<contactref element="C_NRST1" pad="1"/>
+<contactref element="B2" pad="4"/>
+<wire x1="-85.956" y1="-231.555" x2="54.1719" y2="33.707" width="0" layer="19" extent="1-1"/>
+<wire x1="-91.544" y1="-231.555" x2="-85.956" y2="-231.555" width="0" layer="19" extent="1-1"/>
+<wire x1="-91.65" y1="-233.65" x2="-91.544" y2="-231.555" width="0" layer="19" extent="1-1"/>
+</signal>
 </signals>
