File: micromouse-main-board/micromouse-revB/micromouse_board_revB_V0.0.6.brd (EAGLE design)
At the start: 128.4 x 85.5 mm, 117 parts, among them J2 JST_PH, J3 JST_PH, U2 DRV8848PWPR, U6 MPU-6000, X1 RASPI_GPIO_B+#_PIN

Commit message: planes seem to be layed nicely
Parts:
- removed 5V_PWR1, 6V_PWR1: green, micromouse-board-added-piconnector:LED-1206
- removed TP1, TP2, TP3, TP4, TP5, TP6: (no value), micromouse-board-added-piconnector:TESTPOINT_ROUND_2MM
- added 5V_PWR, 6V_PWR: green, micromouse-board-added-piconnector:LED-1206
- added T1, T2, T3, T4, T5, T6, TP12, TP13: (no value), micromouse-board-added-piconnector:TESTPOINT_ROUND_2MM
- R_ERF: value 30 Ohms -> 30
- moved C_NRST1 294.9 mm to (45.6, 22.5), turned to 90 degrees
- moved C_NRST2 288.6 mm to (35.2, 22.1), turned to 90 degrees
- moved B2 282.7 mm to (48.4, 17.6), turned to 180 degrees
- moved B3 282.5 mm to (38.0, 17.6), turned to 180 degrees
- moved NMOS3 11.6 mm to (60.3, 8.92)
- moved C_3.3V6 3.05 mm to (-2.84, 30.8)
- moved U$22 2.98 mm to (-12.4, 63.9)
- moved TP9 2.64 mm to (8.32, 26.2)
- moved TP7 2.15 mm to (8.23, 42.8)
- moved B1 2.11 mm to (34.4, 54.6)
- moved U$16 1.68 mm to (-6.97, 64.0)
- moved C_NRST 1.61 mm to (37.5, 48.2), turned to 0 degrees
- moved C_3.3V7 1.01 mm to (-6.44, 32.7)
- moved TP10 1.01 mm to (8.42, 21.4)
- moved C23 0.90 mm to (69.7, 46.0)
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Connections:
- removed net CURRENT_SENSE: CR1.20
- removed net ENC_LA: CR1.40
- removed net ENC_LB: CR1.39
- removed net ENC_RA: CR1.37
- removed net ENC_RB: CR1.38
- net AGND: now also TP12.P$1
- net GND: now also 5V_PWR.C, 6V_PWR.C, B1.1, TP13.P$1; no longer 5V_PWR1.C, 6V_PWR1.C, TP11.P$1
- net INT: now also CR1.56
- net M1_ENC_A: now also CR1.37
- net M1_ENC_B: now also CR1.38
- net M2_ENC_A: now also CR1.40
- net M2_ENC_B: now also CR1.39
- net MGND: now also TP11.P$1
- net N$14: now also 5V_PWR.A; no longer 5V_PWR1.A
- net N$9: now also 6V_PWR.A; no longer 6V_PWR1.A
- net REC_LD: now also T3.P$1; no longer TP2.P$1
- net REC_LF: now also T1.P$1; no longer TP1.P$1
- net REC_LH: now also T2.P$1; no longer TP4.P$1
- net REC_RD: now also T4.P$1; no longer TP5.P$1
- net REC_RF: now also T6.P$1; no longer TP6.P$1
- net REC_RH: now also T5.P$1; no longer TP3.P$1
- net RESET: now also B1.4
Routing:
- added copper zone on layer 16, net 6V
- added copper zone on layer 1, net GND
Other:
- board text added: "1"
- board text added: "2"
- board text added: "3"
- board text added: "4"
- board text added: "5"
- board text added: "6"
- board text added: "AGND"
- board text added: "BAT 1"
- board text added: "BAT 2"
- board text added: "IMU"
- board text added: "M1 ENC A"
- board text added: "M1 ENC B"
- board text added: "M2 ENC A"
- board text added: "M2 ENC B"
- board text added: "MGND"
- board text added: "MOTOR 1"
- board text added: "MOTOR CTRL"
- board text added: "MOTOR2"
- board text added: "PRGM 1"
- board text added: "PRGM 2"
- board text added: "PWR SWITCh"
- board text added: "Serial Wire"
- board text added: "USART"
