File: micromouse-main-board/micromouse-revB/micromouse_board_revB_V0.0.7.brd (EAGLE design)
At the start: 128.4 x 85.5 mm, 117 parts, among them J2 JST_PH, J3 JST_PH, U2 DRV8848PWPR, U6 MPU-6000, X1 RASPI_GPIO_B+#_PIN

Commit message: planes seem to be layed nicely
Parts:
- removed 5V_PWR1, 6V_PWR1: green, micromouse-board-added-piconnector:LED-1206
- removed TP1, TP2, TP3, TP4, TP5, TP6: (no value), micromouse-board-added-piconnector:TESTPOINT_ROUND_2MM
- added 5V_PWR, 6V_PWR: green, micromouse-board-added-piconnector:LED-1206
- added T1, T2, T3, T4, T5, T6, TP12, TP13: (no value), micromouse-board-added-piconnector:TESTPOINT_ROUND_2MM
- C1: value 0.01uF -> 10nF
- R_ERF: value 30 Ohms -> 30
- moved C_NRST2 293.0 mm to (45.9, 21.8), turned to 90 degrees
- moved C_NRST1 290.0 mm to (35.9, 21.9), turned to 90 degrees
- moved B3 287.0 mm to (48.6, 17.1), turned to 180 degrees
- moved B2 277.7 mm to (38.6, 17.1), turned to 180 degrees
- moved R_RLH 43.2 mm to (87.8, 50.2)
- moved C_5V1 26.1 mm to (-4.48, 38.9), turned to 270 degrees
- moved C_BAT2 14.0 mm to (-13.4, 39.4)
- moved NMOS3 11.6 mm to (60.3, 8.92)
- moved C_BAT1 10.8 mm to (-13.9, 43.9), turned to 90 degrees
- moved R_PWR1 10.4 mm to (-12.9, 32.5)
- moved C_3.3V1 8.79 mm to (-6.33, 11.4)
- moved C_NR 8.66 mm to (-9.96, 15.9), turned to 90 degrees
- moved C22 6.14 mm to (67.5, 40.0)
- moved C2 5.69 mm to (55.0, 43.1)
- moved C23 5.45 mm to (65.4, 41.7), turned to 270 degrees
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Connections:
- removed net CURRENT_SENSE: CR1.20
- removed net ENC_LA: CR1.40
- removed net ENC_LB: CR1.39
- removed net ENC_RA: CR1.37
- removed net ENC_RB: CR1.38
- net 3.3V: no longer C1.2, C8.2, CR1.13
- net A3.3V: now also C1.2, C8.2, CR1.13
- net AGND: now also C1.1, C8.1, CR1.12, TP12.P$1
- net GND: now also 5V_PWR.C, 6V_PWR.C, B1.1, TP13.P$1; no longer 5V_PWR1.C, 6V_PWR1.C, C1.1, C8.1, CR1.12, TP11.P$1
- net INT: now also CR1.56
- net M1_ENC_A: now also CR1.37
- net M1_ENC_B: now also CR1.38
- net M2_ENC_A: now also CR1.40
- net M2_ENC_B: now also CR1.39
- net MGND: now also TP11.P$1
- net N$14: now also 5V_PWR.A; no longer 5V_PWR1.A
- net N$9: now also 6V_PWR.A; no longer 6V_PWR1.A
- net REC_LD: now also T3.P$1; no longer TP2.P$1
- net REC_LF: now also T1.P$1; no longer TP1.P$1
- net REC_LH: now also T2.P$1; no longer TP4.P$1
- net REC_RD: now also T4.P$1; no longer TP5.P$1
- net REC_RF: now also T6.P$1; no longer TP6.P$1
- net REC_RH: now also T5.P$1; no longer TP3.P$1
- net RESET: now also B1.4
Routing:
- net 5V: track 0.00 -> 76.5 mm
- net GND: track 0.00 -> 52.1 mm, vias 0 -> 16
- net D_EM: track 0.00 -> 39.6 mm
- net M1_ENC_A: track 0.00 -> 31.9 mm, vias 0 -> 1
- net M2_ENC_B: track 0.00 -> 30.2 mm, vias 0 -> 1
- net 3.3V: track 0.00 -> 29.1 mm
- net M1_ENC_B: track 0.00 -> 28.4 mm, vias 0 -> 1
- net M2_ENC_A: track 0.00 -> 28.0 mm, vias 0 -> 1
- net REC_RF: track 0.00 -> 27.0 mm
- net REC_RD: track 0.00 -> 25.5 mm
- net REC_RH: track 0.00 -> 21.3 mm
- net BRIDGE_A_2: track 0.00 -> 21.1 mm
- net BRIDGE_A_1: track 0.00 -> 21.0 mm
- net REC_LD: track 0.00 -> 19.8 mm
- net RF_EM: track 0.00 -> 19.7 mm
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- added copper zone on layer 1, net 3.3V
- added copper zone on layer 1, net 5V
- added copper zone on layer 1, net 6V
- added copper zone on layer 1, net GND
- added copper zone on layer 16, net GND
- added copper zone on layer 1, net V_BATT
Other:
- board text added: "1"
- board text added: "2"
- board text added: "3"
- board text added: "4"
- board text added: "5"
- board text added: "6"
- board text added: "AGND"
- board text added: "BAT 1"
- board text added: "BAT 2"
- board text added: "IMU"
- board text added: "L"
- board text added: "M1 ENC A"
- board text added: "M1 ENC B"
- board text added: "M2 ENC A"
- board text added: "M2 ENC B"
- board text added: "MGND"
- board text added: "MOTOR 1"
- board text added: "MOTOR CTRL"
- board text added: "MOTOR2"
- board text added: "OFF"
- board text added: "ON"
- board text added: "PRGM 1"
- board text added: "PRGM 2"
- board text added: "PWR SWITCh"
- board text added: "Serial Wire"
- board text added: "USART"
