File: micromouse-main-board/micromouse-revB/micromouse_board_revB_V0.0.10_B.brd (EAGLE design)
At the start: 128.4 x 85.5 mm, 119 parts, among them J2 JST_PH, J3 JST_PH, U2 DRV8848PWPR, U6 MPU-6000, X1 RASPI_GPIO_B+#_PIN

Commit message: board finalized
Parts:
- moved IMU_C3 23.8 mm to (82.8, 15.1)
- moved R_EH1 17.9 mm to (92.3, 37.9), turned to 0 degrees
- moved NMOS2 10.0 mm to (97.9, 34.6)
- moved IMU_C1 9.38 mm to (74.6, 38.8), turned to 90 degrees
- moved C_EM_D2 8.23 mm to (92.4, 35.5), turned to 0 degrees
- moved R_ED_PD 7.57 mm to (93.1, 40.6), turned to 0 degrees
- moved T4 5.74 mm to (81.7, 23.9)
- moved C_ELF2 4.53 mm to (61.7, 64.8)
- moved R_ED1 4.15 mm to (88.8, 35.4), turned to 180 degrees
- moved R_ELF 3.93 mm to (61.7, 68.5)
- moved R_ELF_PD 3.21 mm to (58.8, 66.8), turned to 90 degrees
- moved C_ELF1 3.17 mm to (64.3, 64.8)
- moved IMU_C2 1.61 mm to (80.2, 36.4), turned to 0 degrees
Connections:
- net USART1_RX: now also X1.8
- net USART1_TX: now also X1.10
Routing:
- net D_EM: track 9.94 -> 40.0 mm
- net REC_RH: track 53.3 -> 29.1 mm
- net H2_EM: track 0.00 -> 16.1 mm
- net H_EM: track 3.12 -> 18.8 mm
- net REC_LH: track 7.65 -> 21.0 mm
- net REC_LD: track 24.1 -> 30.7 mm
- net AGND: track 162.0 -> 156.1 mm, vias 7 -> 5
- net REC_RD: track 35.9 -> 37.5 mm
- net N$28: track 1.32 -> 0.00 mm
- net A3.3V: track 232.5 -> 231.2 mm
- net N$29: track 1.42 -> 2.11 mm
- net I2C_SCL: track 25.3 -> 24.7 mm
- removed copper zone on layer 1, net AGND
