File: micromouse-main-board/micromouse-revB/micromouse_board_revB_V0.0.10_B.sch (EAGLE design)
At the start: 119 parts, among them J2 JST_PH, J3 JST_PH, U2 DRV8848PWPR, U6 MPU-6000, X1 RASPI_GPIO_B+#_PIN

Commit message: board finalized
Connections:
- net USART1_RX: now also X1.TXD
- net USART1_TX: now also X1.RXD
Changed lines of the file:
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@@
 <label x="304.546" y="-33.274" size="1.27" layer="95" xref="yes"/>
+</segment>
+<segment>
+<pinref part="X1" gate="G$1" pin="TXD"/>
+<wire x1="-38.1" y1="200.66" x2="-27.94" y2="200.66" width="0.1524" layer="91"/>
+<label x="-27.94" y="200.66" size="1.27" layer="95" xref="yes"/>
 </segment>
 </net>
@@
 <label x="304.8" y="-35.814" size="1.27" layer="95" xref="yes"/>
 </segment>
+<segment>
+<pinref part="X1" gate="G$1" pin="RXD"/>
+<wire x1="-38.1" y1="198.12" x2="-27.94" y2="198.12" width="0.1524" layer="91"/>
+<label x="-27.94" y="198.12" size="1.27" layer="95" xref="yes"/>
+</segment>
 </net>
