File: micromouse-main-board/micromouse-revB/micromouse_board_revB_V0.0.10_C.brd (EAGLE design)
At the start: 128.4 x 85.5 mm, 119 parts, among them J2 JST_PH, J3 JST_PH, U2 DRV8848PWPR, U6 MPU-6000, X1 RASPI_GPIO_B+#_PIN

Commit message: board finalized
Parts:
- moved R_EH2 29.8 mm to (88.5, 21.2), turned to 90 degrees
- moved C_ERF2 22.3 mm to (93.2, 20.3)
- moved C_E_H2 18.1 mm to (91.1, 20.4)
- moved R_ERF_PD 13.2 mm to (57.6, 10.7)
- moved R_RRH 5.71 mm to (81.3, 15.5)
- moved C_E_H1 4.46 mm to (68.1, 7.05), turned to 0 degrees
- moved C_ERF1 2.65 mm to (68.1, 9.27), turned to 0 degrees
- moved R_ERF 2.08 mm to (62.9, 9.96), turned to 90 degrees
- moved R_EH1 0.87 mm to (86.4, 21.2)
- moved NMOS4 0.81 mm to (83.9, 20.2)
- moved R_RRF 0.33 mm to (64.0, 6.07)
Routing:
- net M2_ENC_B: track 29.0 -> 112.0 mm, vias 1 -> 5
- net M2_ENC_A: track 27.5 -> 105.5 mm, vias 1 -> 5
- net M1_ENC_A: track 37.5 -> 99.6 mm, vias 1 -> 3
- net M1_ENC_B: track 33.0 -> 90.9 mm, vias 1 -> 3
- net NFAULT: track 7.01 -> 52.5 mm, vias 0 -> 6
- net INT: track 4.78 -> 31.1 mm, vias 0 -> 2
- net REC_RF: track 41.6 -> 18.8 mm
- net EM_RF: track 3.31 -> 13.2 mm
- net EM_D: track 3.81 -> 11.9 mm
- net EM_H: track 3.71 -> 11.6 mm
- net EM_LF: track 5.27 -> 12.0 mm
- net 5V: track 27.0 -> 30.1 mm
- net H_EM: track 3.12 -> 0.42 mm
- net N$5: track 0.00 -> 1.72 mm
- net RF_EM: track 19.7 -> 18.1 mm
