File: micromouse-main-board/micromouse-revB/micromouse_board_revB_V0.0.11.sch (EAGLE design)
At the start: 119 parts, among them J2 JST_PH, J3 JST_PH, U2 DRV8848PWPR, U6 MPU-6000, X1 RASPI_GPIO_B+#_PIN

Commit message: board finalized
Connections:
- net I2C_SCL: now also X1.SCL
- net I2C_SDA: now also X1.SDA
Changed lines of the file:
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@@
 <segment>
 <pinref part="X1" gate="G$1" pin="SPI_CE0"/>
-<wire x1="-38.1" y1="208.28" x2="-33.02" y2="208.28" width="0.1524" layer="91"/>
-<label x="-33.02" y="208.28" size="1.27" layer="95" xref="yes"/>
+<wire x1="-38.1" y1="208.28" x2="-27.94" y2="208.28" width="0.1524" layer="91"/>
+<label x="-27.94" y="208.28" size="1.27" layer="95" xref="yes"/>
 </segment>
 </net>
@@
 <segment>
 <pinref part="X1" gate="G$1" pin="SPI_SCLK"/>
-<wire x1="-38.1" y1="210.82" x2="-33.02" y2="210.82" width="0.1524" layer="91"/>
-<label x="-33.02" y="210.82" size="1.27" layer="95" xref="yes"/>
+<wire x1="-38.1" y1="210.82" x2="-27.94" y2="210.82" width="0.1524" layer="91"/>
+<label x="-27.94" y="210.82" size="1.27" layer="95" xref="yes"/>
 </segment>
 </net>
@@
 <segment>
 <pinref part="X1" gate="G$1" pin="SPI_MISO"/>
-<wire x1="-38.1" y1="213.36" x2="-33.02" y2="213.36" width="0.1524" layer="91"/>
-<label x="-33.02" y="213.36" size="1.27" layer="95" xref="yes"/>
+<wire x1="-38.1" y1="213.36" x2="-27.94" y2="213.36" width="0.1524" layer="91"/>
+<label x="-27.94" y="213.36" size="1.27" layer="95" xref="yes"/>
 </segment>
 </net>
@@
 <segment>
 <pinref part="X1" gate="G$1" pin="SPI_MOSI"/>
-<wire x1="-38.1" y1="215.9" x2="-33.02" y2="215.9" width="0.1524" layer="91"/>
-<label x="-33.02" y="215.9" size="1.27" layer="95" xref="yes"/>
+<wire x1="-38.1" y1="215.9" x2="-27.94" y2="215.9" width="0.1524" layer="91"/>
+<label x="-27.94" y="215.9" size="1.27" layer="95" xref="yes"/>
 </segment>
 </net>
@@
 <label x="398.78" y="-190.5" size="1.27" layer="95" rot="R270" xref="yes"/>
 </segment>
+<segment>
+<pinref part="X1" gate="G$1" pin="SDA"/>
+<wire x1="-68.58" y1="165.1" x2="-76.2" y2="165.1" width="0.1524" layer="91"/>
+<label x="-76.2" y="165.1" size="1.27" layer="95" rot="R180" xref="yes"/>
+</segment>
 </net>
 <net name="I2C_SCL" class="0">
@@
 <junction x="124.46" y="-63.246"/>
 </segment>
-</net>
+<segment>
+<pinref part="X1" gate="G$1" pin="SCL"/>
+<wire x1="-68.58" y1="167.64" x2="-76.2" y2="167.64" width="0.1524" layer="91"/>
+<label x="-76.2" y="167.64" size="1.27" layer="95" rot="R180" xref="yes"/>
+</segment>
+</net>
