File: micromouse-main-board/micromouse-revB/micromouse_board_revB_V0.0.12.brd (EAGLE design)
At the start: 128.4 x 85.5 mm, 119 parts, among them J2 JST_PH, J3 JST_PH, U2 DRV8848PWPR, U6 MPU-6000, X1 RASPI_GPIO_B+#_PIN

Commit message: board finalized
Parts:
- moved C_E_H1 47.7 mm to (84.7, 52.0)
- moved C_E_H2 40.6 mm to (84.7, 49.9), turned to 180 degrees
- moved R_EH2 28.5 mm to (87.1, 21.3)
- moved T1 22.4 mm to (56.8, 69.2)
- moved T6 22.2 mm to (59.3, -5.19)
- moved R_EH_PD 14.1 mm to (81.1, 21.0), turned to 270 degrees
- moved C_ELF1 12.3 mm to (72.3, 59.7), turned to 0 degrees
- moved R_ED1 10.8 mm to (94.2, 28.5), turned to 270 degrees
- moved R_ERF_PD 10.3 mm to (60.8, 10.4)
- moved C_ELF2 9.25 mm to (72.3, 61.8), turned to 0 degrees
- moved C_EM_D1 8.79 mm to (94.7, 41.3)
- moved R_RLH 8.62 mm to (79.6, 52.6), turned to 0 degrees
- moved R_ED_PD 8.47 mm to (92.6, 34.8)
- moved NMOS2 8.45 mm to (95.3, 33.0)
- moved R_ERF 7.38 mm to (65.0, 4.47), turned to 270 degrees
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Connections:
- net SPI2_MISO: no longer X1.21
- net SPI2_MOSI: no longer X1.19
- net SPI2_NSS: no longer X1.24
- net SPI2_SCK: no longer X1.23
- net USART1_RX: now also X1.8
- net USART1_TX: now also X1.10
Routing:
- net GND: track 56.8 -> 351.6 mm, vias 34 -> 38
- net USART1_TX: track 27.1 -> 141.2 mm, vias 2 -> 5
- net 5V: track 27.0 -> 137.7 mm, vias 0 -> 1
- net V_BATT: track 25.0 -> 110.9 mm, vias 2 -> 4
- net M2_ENC_B: track 29.0 -> 106.6 mm, vias 1 -> 3
- net M2_ENC_A: track 27.5 -> 104.6 mm, vias 1 -> 3
- net REC_LF: track 21.2 -> 93.6 mm, vias 1 -> 5
- net EM_RF: track 3.31 -> 62.5 mm, vias 0 -> 2
- net M1_ENC_B: track 33.0 -> 91.7 mm, vias 1 -> 3
- net M1_ENC_A: track 37.5 -> 96.1 mm, vias 1 -> 3
- net REC_LH: track 7.65 -> 66.2 mm, vias 0 -> 1
- net AGND: track 162.0 -> 214.6 mm, vias 7 -> 13
- net NFAULT: track 7.01 -> 57.5 mm, vias 0 -> 4
- net 3.3V: track 113.8 -> 163.7 mm
- net EM_H: track 3.71 -> 53.1 mm, vias 0 -> 2
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