File: micromouse-main-board/micromouse-revB/micromouse_board_revB_V0.0.12.sch (EAGLE design)
At the start: 119 parts, among them J2 JST_PH, J3 JST_PH, U2 DRV8848PWPR, U6 MPU-6000, X1 RASPI_GPIO_B+#_PIN

Commit message: board finalized
Connections:
- net SPI2_MISO: no longer X1.SPI_MISO
- net SPI2_MOSI: no longer X1.SPI_MOSI
- net SPI2_NSS: no longer X1.SPI_CE0
- net SPI2_SCK: no longer X1.SPI_SCLK
- net USART1_RX: now also X1.TXD
- net USART1_TX: now also X1.RXD
Changed lines of the file:
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@@
 <label x="474.98" y="-160.02" size="1.27" layer="95" xref="yes"/>
-</segment>
-<segment>
-<pinref part="X1" gate="G$1" pin="SPI_CE0"/>
-<wire x1="-38.1" y1="208.28" x2="-33.02" y2="208.28" width="0.1524" layer="91"/>
-<label x="-33.02" y="208.28" size="1.27" layer="95" xref="yes"/>
 </segment>
 </net>
@@
 <label x="474.98" y="-154.94" size="1.27" layer="95" xref="yes"/>
 </segment>
-<segment>
-<pinref part="X1" gate="G$1" pin="SPI_SCLK"/>
-<wire x1="-38.1" y1="210.82" x2="-33.02" y2="210.82" width="0.1524" layer="91"/>
-<label x="-33.02" y="210.82" size="1.27" layer="95" xref="yes"/>
-</segment>
 </net>
 <net name="SPI2_MISO" class="0">
@@
 <label x="474.98" y="-149.86" size="1.27" layer="95" xref="yes"/>
 </segment>
-<segment>
-<pinref part="X1" gate="G$1" pin="SPI_MISO"/>
-<wire x1="-38.1" y1="213.36" x2="-33.02" y2="213.36" width="0.1524" layer="91"/>
-<label x="-33.02" y="213.36" size="1.27" layer="95" xref="yes"/>
-</segment>
 </net>
 <net name="SPI2_MOSI" class="0">
@@
 <wire x1="462.28" y1="-144.78" x2="474.98" y2="-144.78" width="0.1524" layer="91"/>
 <label x="474.98" y="-144.78" size="1.27" layer="95" xref="yes"/>
-</segment>
-<segment>
-<pinref part="X1" gate="G$1" pin="SPI_MOSI"/>
-<wire x1="-38.1" y1="215.9" x2="-33.02" y2="215.9" width="0.1524" layer="91"/>
-<label x="-33.02" y="215.9" size="1.27" layer="95" xref="yes"/>
 </segment>
 </net>
@@
 <label x="304.546" y="-33.274" size="1.27" layer="95" xref="yes"/>
 </segment>
+<segment>
+<pinref part="X1" gate="G$1" pin="TXD"/>
+<wire x1="-38.1" y1="200.66" x2="-27.94" y2="200.66" width="0.1524" layer="91"/>
+<label x="-27.94" y="200.66" size="1.27" layer="95" xref="yes"/>
+</segment>
 </net>
 <net name="USART1_TX" class="0">
@@
 <label x="304.8" y="-35.814" size="1.27" layer="95" xref="yes"/>
 </segment>
-</net>
+<segment>
+<pinref part="X1" gate="G$1" pin="RXD"/>
+<wire x1="-38.1" y1="198.12" x2="-27.94" y2="198.12" width="0.1524" layer="91"/>
+<label x="-27.94" y="198.12" size="1.27" layer="95" xref="yes"/>
+</segment>
+</net>
