File: micromouse-main-board/micromouse-revB/micromouse_board_revB_V0.0.16.brd (EAGLE design)
At the start: 128.4 x 85.5 mm, 119 parts, among them J2 JST_PH, J3 JST_PH, U2 DRV8848PWPR, U6 MPU-6000, X1 RASPI_GPIO_B+#_PIN

Commit message: board finalized
Parts:
- moved C_E_H1 47.7 mm to (84.7, 52.0)
- moved C_E_H2 40.6 mm to (84.7, 49.9), turned to 180 degrees
- moved R_EH2 28.5 mm to (87.1, 21.3)
- moved T1 22.4 mm to (56.8, 69.2)
- moved T6 22.2 mm to (59.3, -5.19)
- moved R_EH_PD 14.1 mm to (81.1, 21.0), turned to 270 degrees
- moved C_ELF1 12.3 mm to (72.3, 59.7), turned to 0 degrees
- moved R_ED1 10.8 mm to (94.1, 28.5), turned to 270 degrees
- moved R_ERF_PD 10.3 mm to (60.8, 10.4)
- moved C_ELF2 9.25 mm to (72.3, 61.8), turned to 0 degrees
- moved C_EM_D1 8.79 mm to (94.7, 41.3)
- moved R_RLH 8.62 mm to (79.6, 52.6), turned to 0 degrees
- moved R_ED_PD 8.47 mm to (92.6, 34.8)
- moved NMOS2 8.45 mm to (95.3, 33.0)
- moved R_ERF 7.38 mm to (65.0, 4.47), turned to 270 degrees
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Connections:
- net I2C_SCL: now also X1.5
- net I2C_SDA: now also X1.3
Routing:
- net 5V: track 27.0 -> 232.7 mm, vias 0 -> 2
- net AGND: track 162.0 -> 290.0 mm, vias 7 -> 19
- net GND: track 56.8 -> 163.7 mm, vias 34 -> 55
- net I2C_SCL: track 25.3 -> 131.8 mm, vias 0 -> 6
- net SPI2_SCK: track 0.00 -> 104.8 mm, vias 0 -> 1
- net 3.3V: track 113.8 -> 218.4 mm, vias 2 -> 9
- net SPI2_NSS: track 0.00 -> 103.4 mm, vias 0 -> 1
- net SPI2_MISO: track 0.00 -> 92.8 mm, vias 0 -> 1
- net MGND: track 28.0 -> 120.7 mm, vias 0 -> 14
- net SPI2_MOSI: track 0.00 -> 88.8 mm, vias 0 -> 1
- net REC_LF: track 21.2 -> 108.7 mm, vias 1 -> 3
- net A3.3V: track 232.5 -> 319.8 mm, vias 15 -> 22
- net V_BATT: track 25.0 -> 110.9 mm, vias 2 -> 4
- net M2_ENC_B: track 29.0 -> 106.6 mm, vias 1 -> 3
- net M2_ENC_A: track 27.5 -> 104.6 mm, vias 1 -> 3
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- added copper zone on layer 3, net 3.3V
- added copper zone on layer 2, net GND

Commit message: added cam processor and gerbers
Routing:
- net 3.3V: track 218.4 -> 220.4 mm, vias 9 -> 11
Changed lines of the file:
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@@
 <wire x1="52.151" y1="42.499" x2="52.4685" y2="42.1815" width="1.016" layer="1"/>
 <wire x1="54.1719" y1="38.207" x2="53.0352" y2="38.207" width="0.254" layer="1"/>
-<wire x1="55.1704" y1="42.4986" x2="53.1212" y2="42.4986" width="0.762" layer="1"/>
 <wire x1="53.1212" y1="42.4986" x2="52.8041" y2="42.1815" width="0.762" layer="1"/>
 <wire x1="52.8041" y1="42.1815" x2="52.4685" y2="42.1815" width="0.762" layer="1"/>
@@
 <wire x1="-7.1792" y1="9.265" x2="-7.18" y2="9.265" width="1.016" layer="1"/>
 <wire x1="-10.527" y1="11.2164" x2="-10.527" y2="11.4364" width="1.016" layer="1"/>
-<wire x1="-10.527" y1="11.4364" x2="-8.1534" y2="11.4364" width="1.016" layer="1"/>
-<wire x1="-8.1534" y1="11.4364" x2="-7.1792" y2="11.4364" width="1.016" layer="1"/>
+<wire x1="-10.527" y1="11.4364" x2="-7.1792" y2="11.4364" width="1.016" layer="1"/>
 <wire x1="-10.527" y1="11.2164" x2="-10.7706" y2="10.9728" width="0.508" layer="1"/>
 <wire x1="-12.0532" y1="26.7208" x2="-12.0532" y2="25.4898" width="0.508" layer="1"/>
@@
 <wire x1="51.6636" y1="40.3352" x2="52.1002" y2="40.3352" width="0.508" layer="1"/>
 <wire x1="52.1002" y1="40.3352" x2="52.151" y2="40.386" width="0.508" layer="1"/>
+<wire x1="53.1212" y1="42.4986" x2="55.1704" y2="42.4986" width="0.254" layer="1"/>
+<wire x1="55.1704" y1="42.4986" x2="53.896" y2="41.2242" width="0.254" layer="1"/>
+<wire x1="53.896" y1="41.2242" x2="53.6527" y2="41.2242" width="0.254" layer="1"/>
+<via x="53.6527" y="41.2242" extent="1-16" drill="0.35"/>
+<via x="54.6608" y="41.1988" extent="1-16" drill="0.35"/>
 </signal>
 <signal name="V_BATT" class="4">

Commit message: added complete bom, modified board parts based on part availability
Parts:
- R4, R5: value 4.6k -> 4.7k
- R_ERF: value 30 -> 10
- R_PWR1, R_PWR3, R_PWR4: value 100 Ohm -> 150 Ohm
- R_VM1: value 70k -> 75k
- R_VM2: value 40k -> 50k
Changed lines of the file:
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@@
 <attribute name="VALUE" x="58.544" y="66.5012" size="0.4064" layer="27" font="vector"/>
 </element>
-<element name="R_ERF" library="micromouse-board-added-piconnector" library_urn="urn:adsk.eagle:library:14781578" package="0603-RES" package3d_urn="urn:adsk.eagle:package:14781740/2" value="30 " x="64.9616" y="4.4718" smashed="yes" rot="R270">
+<element name="R_ERF" library="micromouse-board-added-piconnector" library_urn="urn:adsk.eagle:library:14781578" package="0603-RES" package3d_urn="urn:adsk.eagle:package:14781740/2" value="10" x="64.9616" y="4.4718" smashed="yes" rot="R270">
 <attribute name="VALUE" x="66.1686" y="5.7378" size="0.4064" layer="27" font="vector" rot="R270"/>
 </element>
@@
 <attribute name="VALUE" x="58.357" y="58.735" size="0.6096" layer="27" font="vector" ratio="20" rot="R180"/>
 </element>
-<element name="R_VM1" library="micromouse-board-added-piconnector" library_urn="urn:adsk.eagle:library:14781578" package="0603-RES" package3d_urn="urn:adsk.eagle:package:14781740/2" value="70k" x="54.4376" y="21.9964" smashed="yes" rot="R90">
+<element name="R_VM1" library="micromouse-board-added-piconnector" library_urn="urn:adsk.eagle:library:14781578" package="0603-RES" package3d_urn="urn:adsk.eagle:package:14781740/2" value="75k" x="54.4376" y="21.9964" smashed="yes" rot="R90">
 <attribute name="VALUE" x="55.9806" y="21.4804" size="0.4064" layer="27" font="vector" rot="R90"/>
 </element>
-<element name="R_VM2" library="micromouse-board-added-piconnector" library_urn="urn:adsk.eagle:library:14781578" package="0603-RES" package3d_urn="urn:adsk.eagle:package:14781740/2" value="40k" x="55.2516" y="19.1568" smashed="yes" rot="R180">
+<element name="R_VM2" library="micromouse-board-added-piconnector" library_urn="urn:adsk.eagle:library:14781578" package="0603-RES" package3d_urn="urn:adsk.eagle:package:14781740/2" value="50k" x="55.2516" y="19.1568" smashed="yes" rot="R180">
 <attribute name="VALUE" x="55.6216" y="20.6938" size="0.4064" layer="27" font="vector" rot="R180"/>
 </element>
@@
 </element>
 <element name="X1" library="raspberrypi_bastelstube_v13" package="RASPI_GPIO_B+_PIN" value="RASPI_GPIO_B+#_PIN" x="-18" y="34.3" smashed="yes" rot="R90"/>
-<element name="R4" library="rcl" library_urn="urn:adsk.eagle:library:334" package="M0805" package3d_urn="urn:adsk.eagle:package:23556/2" value="4.6k" x="49.312" y="19.6048" smashed="yes" rot="R90">
+<element name="R4" library="rcl" library_urn="urn:adsk.eagle:library:334" package="M0805" package3d_urn="urn:adsk.eagle:package:23556/2" value="4.7k" x="49.312" y="19.6048" smashed="yes" rot="R90">
 <attribute name="SPICEPREFIX" value="R" x="49.312" y="19.6048" size="1.778" layer="27" rot="R90" display="off"/>
 <attribute name="VALUE" x="49.402" y="21.9188" size="0.4064" layer="27" font="vector" rot="R90"/>
 </element>
-<element name="R5" library="rcl" library_urn="urn:adsk.eagle:library:334" package="M0805" package3d_urn="urn:adsk.eagle:package:23556/2" value="4.6k" x="47.2218" y="19.5942" smashed="yes" rot="R90">
+<element name="R5" library="rcl" library_urn="urn:adsk.eagle:library:334" package="M0805" package3d_urn="urn:adsk.eagle:package:23556/2" value="4.7k" x="47.2218" y="19.5942" smashed="yes" rot="R90">
 <attribute name="SPICEPREFIX" value="R" x="47.2218" y="19.5942" size="1.778" layer="27" rot="R90" display="off"/>
 <attribute name="VALUE" x="47.4558" y="21.9082" size="0.4064" layer="27" font="vector" rot="R90"/>
@@
 <attribute name="NAME" x="-14.9048" y="24.6134" size="0.8128" layer="25" font="vector" ratio="20"/>
 </element>
-<element name="R_PWR3" library="micromouse-board-added-piconnector" library_urn="urn:adsk.eagle:library:14781578" package="0603-RES" package3d_urn="urn:adsk.eagle:package:14781740/2" value="100 Ohm" x="-12.9548" y="20.974" smashed="yes">
+<element name="R_PWR3" library="micromouse-board-added-piconnector" library_urn="urn:adsk.eagle:library:14781578" package="0603-RES" package3d_urn="urn:adsk.eagle:package:14781740/2" value="150 Ohm" x="-12.9548" y="20.974" smashed="yes">
 <attribute name="VALUE" x="-14.0708" y="19.4818" size="0.4064" layer="27" font="vector"/>
 </element>
@@
 <attribute name="NAME" x="-14.9818" y="30.4808" size="0.8128" layer="25" font="vector" ratio="20"/>
 </element>
-<element name="R_PWR4" library="micromouse-board-added-piconnector" library_urn="urn:adsk.eagle:library:14781578" package="0603-RES" package3d_urn="urn:adsk.eagle:package:14781740/2" value="100 Ohm" x="-12.9032" y="26.7208" smashed="yes">
+<element name="R_PWR4" library="micromouse-board-added-piconnector" library_urn="urn:adsk.eagle:library:14781578" package="0603-RES" package3d_urn="urn:adsk.eagle:package:14781740/2" value="150 Ohm" x="-12.9032" y="26.7208" smashed="yes">
 <attribute name="VALUE" x="-11.2268" y="27.2606" size="0.4064" layer="27" font="vector"/>
 </element>
@@
 <attribute name="NAME" x="-14.8302" y="36.1204" size="0.8128" layer="25" font="vector" ratio="20"/>
 </element>
-<element name="R_PWR1" library="micromouse-board-added-piconnector" library_urn="urn:adsk.eagle:library:14781578" package="0603-RES" package3d_urn="urn:adsk.eagle:package:14781740/2" value="100 Ohm" x="-12.8778" y="32.5374" smashed="yes">
+<element name="R_PWR1" library="micromouse-board-added-piconnector" library_urn="urn:adsk.eagle:library:14781578" package="0603-RES" package3d_urn="urn:adsk.eagle:package:14781740/2" value="150 Ohm" x="-12.8778" y="32.5374" smashed="yes">
 <attribute name="VALUE" x="-11.2038" y="32.816" size="0.4064" layer="27" font="vector"/>
 </element>
